File: Examples/bridgerectifier/bridgerectifier.sch (KiCad schematic (older format))
At the start: 6 parts

Commit message: Modified Example
Parts:
- D1, D2, D3, D4: symbol D -> D-RESCUE-bridgerectifier
- R1: value 1000 -> 1k
Connections:
- net labels added: in1, in2, out
- wire segments 18 -> 21
Changed lines of the file:
@@
 EESchema Schematic File Version 2
+LIBS:eSim_Analog
+LIBS:eSim_Devices
+LIBS:eSim_Digital
+LIBS:eSim_Hybrid
+LIBS:eSim_Miscellaneous
+LIBS:eSim_Sources
+LIBS:eSim_Subckt
+LIBS:eSim_User
+LIBS:bridgerectifier-rescue
 LIBS:power
 LIBS:device
@@
 LIBS:contrib
 LIBS:valves
-LIBS:eSim_Analog
-LIBS:eSim_Devices
-LIBS:eSim_Digital
-LIBS:eSim_Hybrid
-LIBS:eSim_Sources
 LIBS:bridgerectifier-cache
 EELAYER 25 0
@@
 $EndDescr
 $Comp
-L D D1
+L D-RESCUE-bridgerectifier D1
 U 1 1 557F721F
 P 4000 3000
@@
 $EndComp
 $Comp
-L D D3
+L D-RESCUE-bridgerectifier D3
 U 1 1 557F72FE
 P 4950 3000
@@
 $EndComp
 $Comp
-L D D4
+L D-RESCUE-bridgerectifier D4
 U 1 1 557F7345
 P 4950 4400
@@
 $EndComp
 $Comp
-L D D2
+L D-RESCUE-bridgerectifier D2
 U 1 1 557F745E
 P 4000 4400
@@
 $EndComp
 $Comp
-L R R1
-U 1 1 557F76BB
-P 5550 3600
-F 0 "R1" V 5630 3600 50  0000 C CNN
-F 1 "1000" V 5550 3600 50  0000 C CNN
-F 2 "" V 5480 3600 30  0000 C CNN
-F 3 "" H 5550 3600 30  0000 C CNN
-	1    5550 3600
-	1    0    0    -1
-$EndComp
-$Comp
-L GND #PWR01
+L GND-RESCUE-bridgerectifier #PWR01
 U 1 1 557F76F4
 P 5400 5300
@@
 Wire Wire Line
 	4000 4750 5550 4750
-Connection ~ 5400 5300
 Connection ~ 5400 4750
 Wire Wire Line
@@
 	1    0    0    -1
 $EndComp
+$Comp
+L R R1
+U 1 1 55D44082
+P 5500 3550
+F 0 "R1" H 5550 3680 50  0000 C CNN
+F 1 "1k" H 5550 3600 50  0000 C CNN
+F 2 "" H 5550 3530 30  0000 C CNN
+F 3 "" V 5550 3600 30  0000 C CNN
+	1    5500 3550
+	0    1    1    0
+$EndComp
+Text GLabel 5700 2850 2    60   Input ~ 0
+out
+Text GLabel 3550 3000 1    60   Input ~ 0
+in1
+Text GLabel 3850 3900 3    60   Input ~ 0
+in2
+Wire Wire Line
+	3550 3000 3550 3150
+Connection ~ 3550 3150
+Wire Wire Line
+	3850 3900 3850 3750
+Connection ~ 3850 3750
+Wire Wire Line
+	5700 2850 5550 2850
+Connection ~ 5550 2850
 $EndSCHEMATC
