File: Examples/rc/rc.sch (KiCad schematic (older format))
At the start: 3 parts

Commit message: Modified Example
Parts:
- R1: symbol R -> R-RESCUE-rc
Connections:
- net out: now reaches C1.1, R1.1
- net in: now reaches R1.2, v1.1 (+)
Changed lines of the file:
@@
 EESchema Schematic File Version 2
+LIBS:eSim_Analog
+LIBS:eSim_Devices
+LIBS:eSim_Digital
+LIBS:eSim_Hybrid
+LIBS:eSim_Miscellaneous
+LIBS:eSim_Sources
+LIBS:eSim_Subckt
+LIBS:eSim_User
+LIBS:rc-rescue
 LIBS:power
 LIBS:device
@@
 LIBS:memory
 LIBS:xilinx
-LIBS:special
 LIBS:microcontrollers
 LIBS:dsp
@@
 LIBS:contrib
 LIBS:valves
-LIBS:eSim_Analog
-LIBS:eSim_Devices
-LIBS:eSim_Digital
-LIBS:eSim_Hybrid
-LIBS:eSim_Sources
 LIBS:rc-cache
 EELAYER 25 0
@@
 $EndDescr
 $Comp
-L R R1
+L R-RESCUE-rc R1
 U 1 1 556C372A
 P 5100 2300
@@
 	1    0    0    -1
 $EndComp
-Text GLabel 5050 3400 0    60   Input ~ 0
-gnd
 Wire Wire Line
 	4650 2400 4650 2300
@@
 	5600 3300 4650 3300
 Connection ~ 5150 3300
-Wire Wire Line
-	5050 3400 5100 3400
-Wire Wire Line
-	5100 3400 5100 3350
-Wire Wire Line
-	5100 3350 5150 3350
-Connection ~ 5150 3350
 Wire Wire Line
 	5600 2300 5600 2500
@@
 $EndComp
 $Comp
-L GND #PWR?
+L GND-RESCUE-rc #PWR02
 U 1 1 55796439
 P 5150 3400
-F 0 "#PWR?" H 5150 3400 30  0001 C CNN
+F 0 "#PWR02" H 5150 3400 30  0001 C CNN
 F 1 "GND" H 5150 3330 30  0001 C CNN
 F 2 "" H 5150 3400 60  0000 C CNN
@@
 Wire Wire Line
 	5150 3300 5150 3400
+Text GLabel 4600 2250 0    60   Input ~ 0
+in
+Text GLabel 5600 2200 2    60   Input ~ 0
+out
+Wire Wire Line
+	5600 2200 5550 2200
+Wire Wire Line
+	5550 2200 5550 2300
+Connection ~ 5550 2300
+Wire Wire Line
+	4600 2250 4700 2250
+Wire Wire Line
+	4700 2250 4700 2300
+Connection ~ 4700 2300
 $EndSCHEMATC
