File: Examples/BasicGates/BasicGates.sch (KiCad schematic (older format))
At the start: 13 parts, among them U1 adc_bridge_2, U2 d_and, U3 d_or, U4 d_nor, U5 d_nand, U6 d_inverter, U7 d_xor, U8 dac_bridge_1

Commit message: Modified Example
Connections:
- net labels added: IN1, IN2, OUT
- wire segments 65 -> 68
Changed lines of the file:
@@
 EESchema Schematic File Version 2
+LIBS:BasicGates-rescue
 LIBS:power
 LIBS:device
@@
 LIBS:memory
 LIBS:xilinx
-LIBS:special
 LIBS:microcontrollers
 LIBS:dsp
@@
 A
 $Comp
-L GND #PWR01
+L GND-RESCUE-BasicGates #PWR01
 U 1 1 5072534B
 P 10850 3900
@@
 $EndComp
 $Comp
-L GND #PWR03
+L GND-RESCUE-BasicGates #PWR03
 U 1 1 507251E5
 P 2050 1250
@@
 $EndComp
 $Comp
-L GND #PWR04
+L GND-RESCUE-BasicGates #PWR04
 U 1 1 505C9EE8
 P 1650 5900
@@
 	1    0    0    -1
 $EndComp
+Text GLabel 2200 2950 2    60   Input ~ 0
+IN2
+Text GLabel 2250 3450 2    60   Input ~ 0
+IN1
 Wire Wire Line
 	1650 4500 2200 4500
@@
 Wire Wire Line
 	10850 3000 10850 3200
+Wire Wire Line
+	2200 2950 2050 2950
+Connection ~ 2050 2950
+Wire Wire Line
+	2250 3450 2050 3450
+Connection ~ 2050 3450
+Text GLabel 10700 2800 1    60   Input ~ 0
+OUT
+Wire Wire Line
+	10700 2800 10700 3000
+Connection ~ 10700 3000
 $EndSCHEMATC

Commit message: Remove unwanted example
Parts:
- added U10, U11, U9: plot_v1, symbol plot_v1
- R1, R2, R3: symbol R -> R-RESCUE-BasicGates
Connections:
- net OUT: now also U11.~
- net IN1 renamed B
- net B: now also U10.~
- net IN2 renamed A
- net A: now also U9.~
Changed lines of the file:
@@
 EESchema Schematic File Version 2
 LIBS:BasicGates-rescue
+LIBS:eSim_Analog
+LIBS:eSim_Devices
+LIBS:eSim_Digital
+LIBS:eSim_Hybrid
+LIBS:eSim_Miscellaneous
+LIBS:eSim_Plot
+LIBS:eSim_Power
+LIBS:eSim_Sources
+LIBS:eSim_Subckt
+LIBS:eSim_User
 LIBS:power
 LIBS:device
@@
 LIBS:contrib
 LIBS:valves
-LIBS:eSim_Analog
-LIBS:eSim_Devices
-LIBS:eSim_Digital
-LIBS:eSim_Hybrid
-LIBS:eSim_Sources
 LIBS:BasicGates-cache
 EELAYER 25 0
@@
 $EndComp
 $Comp
-L R R3
+L R-RESCUE-BasicGates R3
 U 1 1 507251A7
 P 1400 2200
@@
 $EndComp
 $Comp
-L R R2
+L R-RESCUE-BasicGates R2
 U 1 1 50652FB6
 P 10850 3350
@@
 $EndComp
 $Comp
-L R R1
+L R-RESCUE-BasicGates R1
 U 1 1 505C9F25
 P 2200 5100
@@
 F 3 "" H 2050 2150 60  0000 C CNN
 	1    2050 2150
-	-1   0    0    1
+	1    0    0    1
 $EndComp
 $Comp
@@
 $EndComp
 Text GLabel 2200 2950 2    60   Input ~ 0
-IN2
+A
 Text GLabel 2250 3450 2    60   Input ~ 0
-IN1
+B
 Wire Wire Line
 	1650 4500 2200 4500
@@
 Wire Wire Line
 	3650 1700 3650 2200
-Connection ~ 1400 2750
 Connection ~ 1800 1500
 Wire Wire Line
@@
 	2050 3150 2250 3150
 Wire Wire Line
-	1400 2750 2050 2750
+	1400 2750 2350 2750
 Connection ~ 2050 2750
 Wire Wire Line
@@
 	2250 3450 2050 3450
 Connection ~ 2050 3450
-Text GLabel 10700 2800 1    60   Input ~ 0
+Text GLabel 10850 2800 2    60   Input ~ 0
 OUT
 Wire Wire Line
-	10700 2800 10700 3000
+	10700 2700 10700 3000
 Connection ~ 10700 3000
+$Comp
+L plot_v1 U9
+U 1 1 56D473A0
+P 2350 2900
+F 0 "U9" H 2350 3400 60  0000 C CNN
+F 1 "plot_v1" H 2550 3250 60  0000 C CNN
+F 2 "" H 2350 2900 60  0000 C CNN
+F 3 "" H 2350 2900 60  0000 C CNN
+	1    2350 2900
+	1    0    0    -1
+$EndComp
+$Comp
+L plot_v1 U10
+U 1 1 56D4742D
+P 2350 4400
+F 0 "U10" H 2350 4900 60  0000 C CNN
+F 1 "plot_v1" H 2550 4750 60  0000 C CNN
+F 2 "" H 2350 4400 60  0000 C CNN
+F 3 "" H 2350 4400 60  0000 C CNN
+	1    2350 4400
+	1    0    0    -1
+$EndComp
+$Comp
+L plot_v1 U11
+U 1 1 56D47776
+P 10700 2900
+F 0 "U11" H 10700 3400 60  0000 C CNN
+F 1 "plot_v1" H 10900 3250 60  0000 C CNN
+F 2 "" H 10700 2900 60  0000 C CNN
+F 3 "" H 10700 2900 60  0000 C CNN
+	1    10700 2900
+	1    0    0    -1
+$EndComp
+Wire Wire Line
+	2350 2750 2350 2700
+Wire Wire Line
+	2350 4200 2050 4200
+Connection ~ 2050 4200
+Wire Wire Line
+	10850 2800 10700 2800
+Connection ~ 10700 2800
 $EndSCHEMATC
