File: Examples/HalfAdder/HalfAdder.sch (KiCad schematic (older format))
At the start: 11 parts, among them U1 adc_bridge_2, U2 dac_bridge_2, U3 plot_v1, U4 plot_v1, U5 plot_v1, U6 plot_v1, X1 half_adder

Commit message: Half adder subcircuit filename conflict in Windows
Replaced Half_Adder example with renamed HalfAdder to avoid Windows
case-only filename difference conflict with subcircuit half_adder.
Parts:
- v1, v2: value DC -> PULSE
Changed lines of the file:
@@
 LIBS:eSim_Subckt
 LIBS:eSim_User
-LIBS:Half_Adder-rescue
+LIBS:HalfAdder-rescue
 LIBS:power
 LIBS:device
@@
 LIBS:valves
 LIBS:eSim_Power
-LIBS:Half_Adder-cache
+LIBS:HalfAdder-cache
 EELAYER 25 0
 EELAYER END
@@
 P 3450 3150
 F 0 "v1" H 3250 3250 60  0000 C CNN
-F 1 "DC" H 3250 3100 60  0000 C CNN
+F 1 "PULSE" H 3250 3100 60  0000 C CNN
 F 2 "R1" H 3150 3150 60  0000 C CNN
 F 3 "" H 3450 3150 60  0000 C CNN
@@
 P 3450 3800
 F 0 "v2" H 3250 3900 60  0000 C CNN
-F 1 "DC" H 3250 3750 60  0000 C CNN
+F 1 "PULSE" H 3250 3750 60  0000 C CNN
 F 2 "R1" H 3150 3800 60  0000 C CNN
 F 3 "" H 3450 3800 60  0000 C CNN
@@
 $EndComp
 $Comp
-L GND-RESCUE-Half_Adder #PWR01
+L GND-RESCUE-HalfAdder #PWR01
 U 1 1 558A93BB
 P 2950 4000
@@
 $EndComp
 $Comp
-L GND-RESCUE-Half_Adder #PWR02
+L GND-RESCUE-HalfAdder #PWR02
 U 1 1 558A93D7
 P 2950 3250
@@
 $EndComp
 $Comp
-L GND-RESCUE-Half_Adder #PWR03
+L GND-RESCUE-HalfAdder #PWR03
 U 1 1 558A9480
 P 8350 3650
