File: Examples/4_bit_JK_ff/4_bit_JK_ff.sch (KiCad schematic (older format))
At the start: 25 parts, among them U1 adc_bridge_3, U10 d_jkff, U2 adc_bridge_4, U3 d_jkff, U4 adc_bridge_4, U5 d_jkff, U6 d_and, U7 d_jkff, U8 d_and, U9 dac_bridge_4

Commit message: Modified Example
Parts:
- added U11: dac_bridge_1, symbol dac_bridge_1
Connections:
- net labels added: D1, D2, D3, D4, IN
- wire segments 138 -> 143

Commit message: Remove unwanted example
Parts:
- added U12, U13, U14, U15: plot_v1, symbol plot_v1
- v1, v3: value dc -> DC; symbol dc -> dc-RESCUE-4_bit_JK_ff
- v10, v11, v4, v5, v6, v7, v8, v9: symbol dc -> dc-RESCUE-4_bit_JK_ff
Connections:
- wire segments 143 -> 144
Other:
- moved on the sheet: R1, R2, R3, R4
Changed lines of the file:
@@
 EESchema Schematic File Version 2
+LIBS:4_bit_JK_ff-rescue
 LIBS:eSim_Analog
 LIBS:eSim_Devices
@@
 LIBS:eSim_Hybrid
 LIBS:eSim_Miscellaneous
+LIBS:eSim_Plot
+LIBS:eSim_Power
 LIBS:eSim_Sources
 LIBS:eSim_Subckt
 LIBS:eSim_User
-LIBS:4_bit_JK_ff-rescue
 LIBS:power
 LIBS:device
@@
 $EndComp
 $Comp
-L dc v1
+L dc-RESCUE-4_bit_JK_ff v1
 U 1 1 5548DFB1
 P 1100 5600
 F 0 "v1" H 900 5700 60  0000 C CNN
-F 1 "dc" H 900 5550 60  0000 C CNN
+F 1 "DC" H 900 5550 60  0000 C CNN
 F 2 "R1" H 800 5600 60  0000 C CNN
 F 3 "" H 1100 5600 60  0000 C CNN
@@
 $EndComp
 $Comp
-L dc v3
+L dc-RESCUE-4_bit_JK_ff v3
 U 1 1 5548E056
 P 1100 6800
 F 0 "v3" H 900 6900 60  0000 C CNN
-F 1 "dc" H 900 6750 60  0000 C CNN
+F 1 "DC" H 900 6750 60  0000 C CNN
 F 2 "R1" H 800 6800 60  0000 C CNN
 F 3 "" H 1100 6800 60  0000 C CNN
@@
 $EndComp
 $Comp
-L dc v4
+L dc-RESCUE-4_bit_JK_ff v4
 U 1 1 554A0BE0
 P 3550 5950
@@
 $EndComp
 $Comp
-L dc v10
+L dc-RESCUE-4_bit_JK_ff v10
 U 1 1 554B724D
 P 3500 6400
@@
 $EndComp
 $Comp
-L dc v11
+L dc-RESCUE-4_bit_JK_ff v11
 U 1 1 554B72DB
 P 3500 6700
@@
 $EndComp
 $Comp
-L dc v9
+L dc-RESCUE-4_bit_JK_ff v9
 U 1 1 554B7321
 P 3500 5450
@@
 $EndComp
 $Comp
-L dc v8
+L dc-RESCUE-4_bit_JK_ff v8
 U 1 1 554B79B1
 P 2200 1200
@@
 $EndComp
 $Comp
-L dc v6
+L dc-RESCUE-4_bit_JK_ff v6
 U 1 1 554B79BD
 P 2150 1650
@@
 $EndComp
 $Comp
-L dc v7
+L dc-RESCUE-4_bit_JK_ff v7
 U 1 1 554B79C3
 P 2150 1950
@@
 $EndComp
 $Comp
-L dc v5
+L dc-RESCUE-4_bit_JK_ff v5
 U 1 1 554B79C9
 P 2150 700
@@
 L GND-RESCUE-4_bit_JK_ff #PWR02
 U 1 1 554B90FC
-P 10450 2400
-F 0 "#PWR02" H 10450 2150 50  0001 C CNN
-F 1 "GND" H 10450 2250 50  0000 C CNN
-F 2 "" H 10450 2400 60  0000 C CNN
-F 3 "" H 10450 2400 60  0000 C CNN
-	1    10450 2400
+P 10850 2400
+F 0 "#PWR02" H 10850 2150 50  0001 C CNN
+F 1 "GND" H 10850 2250 50  0000 C CNN
+F 2 "" H 10850 2400 60  0000 C CNN
+F 3 "" H 10850 2400 60  0000 C CNN
+	1    10850 2400
 	1    0    0    -1
 $EndComp
@@
 	9300 1950 9300 1800
 Wire Wire Line
-	9300 1800 9800 1800
+	9300 1800 10200 1800
 Wire Wire Line
 	9100 2050 9500 2050
@@
 	9500 2050 9500 1950
 Wire Wire Line
-	9500 1950 9800 1950
+	9500 1950 10200 1950
 Wire Wire Line
 	9100 2150 9700 2150
@@
 	9700 2150 9700 2100
 Wire Wire Line
-	9700 2100 9800 2100
-Wire Wire Line
-	9100 2250 9800 2250
-Wire Wire Line
-	10100 1800 10450 1800
-Wire Wire Line
-	10450 1800 10450 2400
-Wire Wire Line
-	10100 1950 10450 1950
-Connection ~ 10450 1950
-Wire Wire Line
-	10100 2100 10450 2100
-Connection ~ 10450 2100
-Wire Wire Line
-	10100 2250 10450 2250
-Connection ~ 10450 2250
+	9700 2100 10200 2100
+Wire Wire Line
+	9100 2250 10200 2250
+Wire Wire Line
+	10500 1800 10850 1800
+Wire Wire Line
+	10850 1800 10850 2400
+Wire Wire Line
+	10500 1950 10850 1950
+Connection ~ 10850 1950
+Wire Wire Line
+	10500 2100 10850 2100
+Connection ~ 10850 2100
+Wire Wire Line
+	10500 2250 10850 2250
+Connection ~ 10850 2250
 Wire Wire Line
 	3050 5450 2800 5450
@@
 L R R1
 U 1 1 55D466F5
-P 9900 1850
-F 0 "R1" H 9950 1980 50  0000 C CNN
-F 1 "1k" H 9950 1900 50  0000 C CNN
-F 2 "" H 9950 1830 30  0000 C CNN
-F 3 "" V 9950 1900 30  0000 C CNN
-	1    9900 1850
+P 10300 1850
+F 0 "R1" H 10350 1980 50  0000 C CNN
+F 1 "1k" H 10350 1900 50  0000 C CNN
+F 2 "" H 10350 1830 30  0000 C CNN
+F 3 "" V 10350 1900 30  0000 C CNN
+	1    10300 1850
 	1    0    0    -1
 $EndComp
@@
 L R R2
 U 1 1 55D46764
-P 9900 2000
-F 0 "R2" H 9950 2130 50  0000 C CNN
-F 1 "1k" H 9950 2050 50  0000 C CNN
-F 2 "" H 9950 1980 30  0000 C CNN
-F 3 "" V 9950 2050 30  0000 C CNN
-	1    9900 2000
+P 10300 2000
+F 0 "R2" H 10350 2130 50  0000 C CNN
+F 1 "1k" H 10350 2050 50  0000 C CNN
+F 2 "" H 10350 1980 30  0000 C CNN
+F 3 "" V 10350 2050 30  0000 C CNN
+	1    10300 2000
 	1    0    0    -1
 $EndComp
@@
 L R R3
 U 1 1 55D467C3
-P 9900 2150
-F 0 "R3" H 9950 2280 50  0000 C CNN
-F 1 "1k" H 9950 2200 50  0000 C CNN
-F 2 "" H 9950 2130 30  0000 C CNN
-F 3 "" V 9950 2200 30  0000 C CNN
-	1    9900 2150
+P 10300 2150
+F 0 "R3" H 10350 2280 50  0000 C CNN
+F 1 "1k" H 10350 2200 50  0000 C CNN
+F 2 "" H 10350 2130 30  0000 C CNN
+F 3 "" V 10350 2200 30  0000 C CNN
+	1    10300 2150
 	1    0    0    -1
 $EndComp
@@
 L R R4
 U 1 1 55D4681D
-P 9900 2300
-F 0 "R4" H 9950 2430 50  0000 C CNN
-F 1 "1k" H 9950 2350 50  0000 C CNN
-F 2 "" H 9950 2280 30  0000 C CNN
-F 3 "" V 9950 2350 30  0000 C CNN
-	1    9900 2300
+P 10300 2300
+F 0 "R4" H 10350 2430 50  0000 C CNN
+F 1 "1k" H 10350 2350 50  0000 C CNN
+F 2 "" H 10350 2280 30  0000 C CNN
+F 3 "" V 10350 2350 30  0000 C CNN
+	1    10300 2300
 	1    0    0    -1
 $EndComp
@@
 Wire Wire Line
 	10650 5350 10650 5500
+$Comp
+L plot_v1 U12
+U 1 1 56D836F6
+P 9400 1900
+F 0 "U12" H 9400 2400 60  0000 C CNN
+F 1 "plot_v1" H 9600 2250 60  0000 C CNN
+F 2 "" H 9400 1900 60  0000 C CNN
+F 3 "" H 9400 1900 60  0000 C CNN
+	1    9400 1900
+	1    0    0    -1
+$EndComp
+$Comp
+L plot_v1 U14
+U 1 1 56D837A6
+P 9950 2050
+F 0 "U14" H 9950 2550 60  0000 C CNN
+F 1 "plot_v1" H 10150 2400 60  0000 C CNN
+F 2 "" H 9950 2050 60  0000 C CNN
+F 3 "" H 9950 2050 60  0000 C CNN
+	1    9950 2050
+	1    0    0    1
+$EndComp
+$Comp
+L plot_v1 U15
+U 1 1 56D84035
+P 10000 2300
+F 0 "U15" H 10000 2800 60  0000 C CNN
+F 1 "plot_v1" H 10200 2650 60  0000 C CNN
+F 2 "" H 10000 2300 60  0000 C CNN
+F 3 "" H 10000 2300 60  0000 C CNN
+	1    10000 2300
+	1    0    0    -1
+$EndComp
+$Comp
+L plot_v1 U13
+U 1 1 56D840C8
+P 9700 2150
+F 0 "U13" H 9700 2650 60  0000 C CNN
+F 1 "plot_v1" H 9900 2500 60  0000 C CNN
+F 2 "" H 9700 2150 60  0000 C CNN
+F 3 "" H 9700 2150 60  0000 C CNN
+	1    9700 2150
+	1    0    0    -1
+$EndComp
+Wire Wire Line
+	9400 1700 9400 1800
+Connection ~ 9400 1800
+Connection ~ 9700 1950
+Connection ~ 10000 2100
+Connection ~ 9950 2250
 $EndSCHEMATC

Commit message: common code for Win and Linux, merged py2 changes
Parts:
- R1, R2, R3, R4: symbol R -> R-RESCUE-4_bit_JK_ff
Changed lines of the file:
@@
 Connection ~ 9400 2250
 $Comp
-L R R1
+L R-RESCUE-4_bit_JK_ff R1
 U 1 1 55D466F5
 P 10300 1850
@@
 $EndComp
 $Comp
-L R R2
+L R-RESCUE-4_bit_JK_ff R2
 U 1 1 55D46764
 P 10300 2000
@@
 $EndComp
 $Comp
-L R R3
+L R-RESCUE-4_bit_JK_ff R3
 U 1 1 55D467C3
 P 10300 2150
@@
 $EndComp
 $Comp
-L R R4
+L R-RESCUE-4_bit_JK_ff R4
 U 1 1 55D4681D
 P 10300 2300
