File: Examples/BJT_Biascircuit/BJT_Biascircuit.sch (KiCad schematic (older format))
At the start: 6 parts, among them Q1 NPN, U1 plot_i2

Commit message: common code for Win and Linux, merged py2 changes
Parts:
- removed Q1: NPN, symbol NPN
- added Q1: eSim_NPN, symbol eSim_NPN
- R1, R2: symbol R -> R-RESCUE-BJT_Biascircuit
- v1: symbol DC -> DC-RESCUE-BJT_Biascircuit
Connections:
- net GND: now also Q1.3 (E)
- net at R1.2: now also Q1.1 (C)
- net at R2.1: now also Q1.2 (B)
Changed lines of the file:
@@
 EESchema Schematic File Version 2
+LIBS:BJT_Biascircuit-rescue
 LIBS:eSim_Analog
 LIBS:eSim_Devices
@@
 $EndDescr
 $Comp
-L NPN Q1
-U 1 1 56A86C4C
-P 5350 3200
-F 0 "Q1" H 5250 3250 50  0000 R CNN
-F 1 "NPN" H 5300 3350 50  0000 R CNN
-F 2 "" H 5550 3300 29  0000 C CNN
-F 3 "" H 5350 3200 60  0000 C CNN
-	1    5350 3200
-	1    0    0    -1
-$EndComp
-$Comp
-L DC v1
+L DC-RESCUE-BJT_Biascircuit v1
 U 1 1 56A86D0E
 P 6600 3050
@@
 vce
 $Comp
-L R R1
+L R-RESCUE-BJT_Biascircuit R1
 U 1 1 56C44AD7
 P 5400 2650
@@
 $EndComp
 $Comp
-L R R2
+L R-RESCUE-BJT_Biascircuit R2
 U 1 1 56C44C4B
 P 4800 3150
@@
 	1    0    0    -1
 $EndComp
+$Comp
+L eSim_NPN Q1
+U 1 1 5D5CEC51
+P 5350 3200
+F 0 "Q1" H 5250 3250 50  0000 R CNN
+F 1 "eSim_NPN" H 5300 3350 50  0000 R CNN
+F 2 "" H 5550 3300 29  0000 C CNN
+F 3 "" H 5350 3200 60  0000 C CNN
+	1    5350 3200
+	1    0    0    -1
+$EndComp
+$Comp
+L PWR_FLAG #FLG02
+U 1 1 5D665114
+P 5600 4150
+F 0 "#FLG02" H 5600 4225 50  0001 C CNN
+F 1 "PWR_FLAG" H 5600 4300 50  0000 C CNN
+F 2 "" H 5600 4150 50  0001 C CNN
+F 3 "" H 5600 4150 50  0001 C CNN
+	1    5600 4150
+	1    0    0    -1
+$EndComp
+Wire Wire Line
+	5600 4150 5600 4250
+Connection ~ 5600 4250
 $EndSCHEMATC
