File: Examples/BJT_CB_config/BJT_CB_config.sch (KiCad schematic (older format))
At the start: 6 parts, among them Q1 NPN

Commit message: common code for Win and Linux, merged py2 changes
Parts:
- removed Q1: NPN, symbol NPN
- added Q1: eSim_NPN, symbol eSim_NPN
- R1, R2: symbol R -> R-RESCUE-BJT_CB_config
- v1: symbol DC -> DC-RESCUE-BJT_CB_config
Connections:
- net GND: now also Q1.2 (B)
- net at R1.2: now also Q1.1 (C)
- net at R2.1: now also Q1.3 (E)
Changed lines of the file:
@@
 EESchema Schematic File Version 2
+LIBS:BJT_CB_config-rescue
 LIBS:eSim_Analog
 LIBS:eSim_Devices
@@
 $EndDescr
 $Comp
-L NPN Q1
-U 1 1 56A86C4C
-P 5450 3200
-F 0 "Q1" H 5350 3250 50  0000 R CNN
-F 1 "NPN" H 5400 3350 50  0000 R CNN
-F 2 "" H 5650 3300 29  0000 C CNN
-F 3 "" H 5450 3200 60  0000 C CNN
-	1    5450 3200
-	0    1    -1   0
-$EndComp
-$Comp
-L DC v1
+L DC-RESCUE-BJT_CB_config v1
 U 1 1 56A86D0E
 P 6600 3050
@@
 vcb
 $Comp
-L R R1
+L R-RESCUE-BJT_CB_config R1
 U 1 1 56C44AD7
 P 5600 2750
@@
 $EndComp
 $Comp
-L R R2
+L R-RESCUE-BJT_CB_config R2
 U 1 1 56C44C4B
 P 4900 3050
@@
 	1    0    0    -1
 $EndComp
+$Comp
+L eSim_NPN Q1
+U 1 1 5D5CEEB2
+P 5450 3200
+F 0 "Q1" H 5350 3250 50  0000 R CNN
+F 1 "eSim_NPN" H 5400 3350 50  0000 R CNN
+F 2 "" H 5650 3300 29  0000 C CNN
+F 3 "" H 5450 3200 60  0000 C CNN
+	1    5450 3200
+	0    1    -1   0
+$EndComp
+$Comp
+L PWR_FLAG #FLG02
+U 1 1 5D665163
+P 5600 4150
+F 0 "#FLG02" H 5600 4225 50  0001 C CNN
+F 1 "PWR_FLAG" H 5600 4300 50  0000 C CNN
+F 2 "" H 5600 4150 50  0001 C CNN
+F 3 "" H 5600 4150 50  0001 C CNN
+	1    5600 4150
+	1    0    0    -1
+$EndComp
+Wire Wire Line
+	5600 4150 5600 4250
+Connection ~ 5600 4250
 $EndSCHEMATC
