File: Examples/BJT_Frequency_Response/BJT_Frequency_Response.sch (KiCad schematic (older format))
At the start: 15 parts, among them Q1 NPN, U1 plot_v1, U2 plot_phase, U3 plot_log

Commit message: common code for Win and Linux, merged py2 changes
Parts:
- removed Q1: NPN, symbol NPN
- added Q1: eSim_NPN, symbol eSim_NPN
Other:
- moved on the sheet: R1, R2, R3, R4, R5, R6
Changed lines of the file:
@@
 LIBS:eSim_Hybrid
 LIBS:eSim_Miscellaneous
-LIBS:eSim_Plot
 LIBS:eSim_Power
 LIBS:eSim_Sources
 LIBS:eSim_Subckt
 LIBS:eSim_User
+LIBS:eSim_Plot
 LIBS:adc-dac
 LIBS:memory
@@
 LIBS:74xx
 LIBS:cmos4000
-LIBS:CE_Amplifier-cache
+LIBS:BJT_Frequency_Response-cache
 EELAYER 25 0
 EELAYER END
@@
 $EndComp
 $Comp
-L PWR_FLAG #FLG01
-U 1 1 51A48298
-P 5650 4450
-F 0 "#FLG01" H 5650 4720 30  0001 C CNN
-F 1 "PWR_FLAG" H 5650 4680 30  0000 C CNN
-F 2 "" H 5650 4450 60  0001 C CNN
-F 3 "" H 5650 4450 60  0001 C CNN
-	1    5650 4450
-	1    0    0    -1
-$EndComp
-$Comp
 L C C1
 U 1 1 51A47FA0
@@
 	0    1    1    0
 $EndComp
-$Comp
-L NPN Q1
-U 1 1 557583B4
-P 5750 3600
-F 0 "Q1" H 5650 3650 50  0000 R CNN
-F 1 "NPN" H 5700 3750 50  0000 R CNN
-F 2 "" H 5950 3700 29  0000 C CNN
-F 3 "" H 5750 3600 60  0000 C CNN
-	1    5750 3600
-	1    0    0    -1
-$EndComp
 Wire Wire Line
 	6100 2900 6100 2800
@@
 L R R3
 U 1 1 56C1B05C
-P 5050 4150
-F 0 "R3" H 5100 4280 50  0000 C CNN
-F 1 "50k" H 5100 4200 50  0000 C CNN
-F 2 "" H 5100 4130 30  0000 C CNN
-F 3 "" V 5100 4200 30  0000 C CNN
-	1    5050 4150
-	0    1    1    0
+P 5100 4200
+F 0 "R3" H 5150 4330 50  0000 C CNN
+F 1 "50k" H 5150 4250 50  0000 C CNN
+F 2 "" H 5150 4180 30  0000 C CNN
+F 3 "" V 5150 4250 30  0000 C CNN
+	1    5100 4200
+	-1   0    0    1
 $EndComp
 $Comp
 L R R4
 U 1 1 56C1B119
-P 5800 4150
-F 0 "R4" H 5850 4280 50  0000 C CNN
-F 1 "1.5k" H 5850 4200 50  0000 C CNN
-F 2 "" H 5850 4130 30  0000 C CNN
-F 3 "" V 5850 4200 30  0000 C CNN
-	1    5800 4150
-	0    1    1    0
+P 5850 4200
+F 0 "R4" H 5900 4330 50  0000 C CNN
+F 1 "1.5k" H 5900 4250 50  0000 C CNN
+F 2 "" H 5900 4180 30  0000 C CNN
+F 3 "" V 5900 4250 30  0000 C CNN
+	1    5850 4200
+	-1   0    0    1
 $EndComp
 $Comp
 L R R6
 U 1 1 56C1B187
-P 7000 4150
-F 0 "R6" H 7050 4280 50  0000 C CNN
-F 1 "1k" H 7050 4200 50  0000 C CNN
-F 2 "" H 7050 4130 30  0000 C CNN
-F 3 "" V 7050 4200 30  0000 C CNN
-	1    7000 4150
-	0    1    1    0
+P 7050 4200
+F 0 "R6" H 7100 4330 50  0000 C CNN
+F 1 "1k" H 7100 4250 50  0000 C CNN
+F 2 "" H 7100 4180 30  0000 C CNN
+F 3 "" V 7100 4250 30  0000 C CNN
+	1    7050 4200
+	-1   0    0    1
 $EndComp
 $Comp
 L R R5
 U 1 1 56C1B28B
-P 6050 3000
-F 0 "R5" H 6100 3130 50  0000 C CNN
-F 1 "2k" H 6100 3050 50  0000 C CNN
-F 2 "" H 6100 2980 30  0000 C CNN
-F 3 "" V 6100 3050 30  0000 C CNN
-	1    6050 3000
-	0    1    1    0
+P 6100 3050
+F 0 "R5" H 6150 3180 50  0000 C CNN
+F 1 "2k" H 6150 3100 50  0000 C CNN
+F 2 "" H 6150 3030 30  0000 C CNN
+F 3 "" V 6150 3100 30  0000 C CNN
+	1    6100 3050
+	-1   0    0    1
 $EndComp
 $Comp
 L R R2
 U 1 1 56C1B323
-P 5050 3000
-F 0 "R2" H 5100 3130 50  0000 C CNN
-F 1 "200k" H 5100 3050 50  0000 C CNN
-F 2 "" H 5100 2980 30  0000 C CNN
-F 3 "" V 5100 3050 30  0000 C CNN
-	1    5050 3000
-	0    1    1    0
-$EndComp
-$Comp
-L GND #PWR02
+P 5100 3050
+F 0 "R2" H 5150 3180 50  0000 C CNN
+F 1 "200k" H 5150 3100 50  0000 C CNN
+F 2 "" H 5150 3030 30  0000 C CNN
+F 3 "" V 5150 3100 30  0000 C CNN
+	1    5100 3050
+	-1   0    0    1
+$EndComp
+$Comp
+L GND #PWR01
 U 1 1 56C1B4E1
 P 5650 4850
-F 0 "#PWR02" H 5650 4600 50  0001 C CNN
+F 0 "#PWR01" H 5650 4600 50  0001 C CNN
 F 1 "GND" H 5650 4700 50  0000 C CNN
 F 2 "" H 5650 4850 50  0000 C CNN
@@
 L R R1
 U 1 1 56C1B3CB
-P 4100 3550
-F 0 "R1" H 4150 3680 50  0000 C CNN
-F 1 "50" H 4150 3600 50  0000 C CNN
-F 2 "" H 4150 3530 30  0000 C CNN
-F 3 "" V 4150 3600 30  0000 C CNN
-	1    4100 3550
-	-1   0    0    1
+P 4050 3600
+F 0 "R1" H 4100 3730 50  0000 C CNN
+F 1 "50" H 4100 3650 50  0000 C CNN
+F 2 "" H 4100 3580 30  0000 C CNN
+F 3 "" V 4100 3650 30  0000 C CNN
+	1    4050 3600
+	0    -1   -1   0
 $EndComp
 $Comp
@@
 	1    0    0    -1
 $EndComp
+$Comp
+L eSim_NPN Q1
+U 1 1 5D5CEEC5
+P 5750 3600
+F 0 "Q1" H 5650 3650 50  0000 R CNN
+F 1 "eSim_NPN" H 5700 3750 50  0000 R CNN
+F 2 "" H 5950 3700 29  0000 C CNN
+F 3 "" H 5750 3600 60  0000 C CNN
+	1    5750 3600
+	1    0    0    -1
+$EndComp
