File: Examples/Clampercircuit/Clampercircuit.sch (KiCad schematic (older format))
At the start: 10 parts, among them U1 plot_v1, U2 plot_v1, U3 plot_v1, U4 plot_v1

Commit message: common code for Win and Linux, merged py2 changes
Parts:
- D1, D2: symbol D -> D-RESCUE-Clampercircuit
Changed lines of the file:
@@
 EESchema Schematic File Version 2
+LIBS:Clampercircuit-rescue
 LIBS:eSim_Analog
 LIBS:eSim_Devices
@@
 $EndComp
 $Comp
-L D D1
+L D-RESCUE-Clampercircuit D1
 U 1 1 56A86555
 P 5100 3400
@@
 $EndComp
 $Comp
-L D D2
+L D-RESCUE-Clampercircuit D2
 U 1 1 56A867F1
 P 8500 3400
