File: Examples/Clippercircuit/Clippercircuit.sch (KiCad schematic (older format))
At the start: 6 parts, among them U1 plot_v1, U2 plot_v1

Commit message: common code for Win and Linux, merged py2 changes
Parts:
- D1, D2: symbol D -> D-RESCUE-Clippercircuit
- R1: symbol R -> R-RESCUE-Clippercircuit
Changed lines of the file:
@@
 EESchema Schematic File Version 2
+LIBS:Clippercircuit-rescue
 LIBS:eSim_Analog
 LIBS:eSim_Devices
@@
 $EndComp
 $Comp
-L D D1
+L D-RESCUE-Clippercircuit D1
 U 1 1 56A86229
 P 5550 3450
@@
 $EndComp
 $Comp
-L D D2
+L D-RESCUE-Clippercircuit D2
 U 1 1 56A863C8
 P 6250 3450
@@
 $EndComp
 $Comp
-L R R1
+L R-RESCUE-Clippercircuit R1
 U 1 1 56A86416
 P 4700 3050
