File: Examples/Diode_characteristics/Diode_characteristics.sch (KiCad schematic (older format))
At the start: 4 parts, among them U1 plot_i2

Commit message: common code for Win and Linux, merged py2 changes
Parts:
- D1: symbol D -> D-RESCUE-Diode_characteristics
- R1: symbol R -> R-RESCUE-Diode_characteristics
- v1: symbol DC -> DC-RESCUE-Diode_characteristics
Changed lines of the file:
@@
 EESchema Schematic File Version 2
+LIBS:Diode_characteristics-rescue
 LIBS:eSim_Analog
 LIBS:eSim_Devices
@@
 $EndDescr
 $Comp
-L DC v1
+L DC-RESCUE-Diode_characteristics v1
 U 1 1 562485DC
 P 4350 3150
@@
 $EndComp
 $Comp
-L D D1
+L D-RESCUE-Diode_characteristics D1
 U 1 1 5624867D
 P 5150 2500
@@
 $EndComp
 $Comp
-L R R1
+L R-RESCUE-Diode_characteristics R1
 U 1 1 562486CA
 P 6900 2950
