File: Examples/FET_Amplifier/FET_Amplifier.sch (KiCad schematic (older format))
At the start: 10 parts, among them J1 NJF, U1 plot_v1, U2 plot_v1

Commit message: common code for Win and Linux, merged py2 changes
Parts:
- removed J1: NJF, symbol NJF
- added J1: eSim_NJF, symbol eSim_NJF
- R2, R3, R4: symbol R -> R-RESCUE-FET_Amplifier
- v2: symbol DC -> DC-RESCUE-FET_Amplifier
Connections:
- wire segments 20 -> 21
Changed lines of the file:
@@
 $EndComp
 $Comp
-L DC v2
+L DC-RESCUE-FET_Amplifier v2
 U 1 1 554CD920
 P 8600 3650
@@
 Connection ~ 5150 4800
 $Comp
-L NJF J1
-U 1 1 557065CE
-P 6200 3500
-F 0 "J1" H 6100 3550 50  0000 R CNN
-F 1 "NJF" H 6150 3650 50  0000 R CNN
-F 2 "" H 6400 3600 29  0000 C CNN
-F 3 "" H 6200 3500 60  0000 C CNN
-	1    6200 3500
-	1    0    0    -1
-$EndComp
-$Comp
-L R R3
+L R-RESCUE-FET_Amplifier R3
 U 1 1 55D44D80
 P 6250 2550
@@
 $EndComp
 $Comp
-L R R2
+L R-RESCUE-FET_Amplifier R2
 U 1 1 55D44EE5
 P 5200 4350
@@
 $EndComp
 $Comp
-L R R4
+L R-RESCUE-FET_Amplifier R4
 U 1 1 55D44F9D
 P 6350 4450
@@
 	3350 3350 3550 3350
 Connection ~ 3550 3350
+$Comp
+L eSim_NJF J1
+U 1 1 5D676189
+P 6200 3500
+F 0 "J1" H 6100 3550 50  0000 R CNN
+F 1 "eSim_NJF" H 6150 3650 50  0000 R CNN
+F 2 "" H 6400 3600 29  0000 C CNN
+F 3 "" H 6200 3500 60  0000 C CNN
+	1    6200 3500
+	1    0    0    -1
+$EndComp
+$Comp
+L PWR_FLAG #FLG02
+U 1 1 5D6762AD
+P 6500 4650
+F 0 "#FLG02" H 6500 4725 50  0001 C CNN
+F 1 "PWR_FLAG" H 6500 4800 50  0000 C CNN
+F 2 "" H 6500 4650 50  0001 C CNN
+F 3 "" H 6500 4650 50  0001 C CNN
+	1    6500 4650
+	1    0    0    -1
+$EndComp
+Wire Wire Line
+	6500 4650 6500 4800
+Connection ~ 6500 4800
 $EndSCHEMATC
