File: Examples/FrequencyResponse_JFET/FrequencyResponse_JFET.sch (KiCad schematic (older format))
At the start: 18 parts, among them J1 NJF, U1 vplot8_1, U2 vplot8_1

Commit message: Modified Example
Parts:
- removed U1, U2: vplot8_1, symbol vplot8_1
Connections:
- net labels added: Out, in
Changed lines of the file:
@@
 EESchema Schematic File Version 2
+LIBS:eSim_Analog
+LIBS:eSim_Devices
+LIBS:eSim_Digital
+LIBS:eSim_Hybrid
+LIBS:eSim_Miscellaneous
+LIBS:eSim_Sources
+LIBS:eSim_Subckt
+LIBS:eSim_User
 LIBS:power
 LIBS:device
@@
 LIBS:memory
 LIBS:xilinx
-LIBS:special
 LIBS:microcontrollers
 LIBS:dsp
@@
 LIBS:contrib
 LIBS:valves
-LIBS:eSim_Analog
-LIBS:eSim_Devices
-LIBS:eSim_Digital
-LIBS:eSim_Hybrid
-LIBS:sourcesSpice
-LIBS:measurementSpice
 LIBS:FrequencyResponse_JFET-cache
 EELAYER 25 0
@@
 $EndDescr
 $Comp
-L R R3
-U 1 1 554CCD03
-P 6300 2600
-F 0 "R3" V 6380 2600 50  0000 C CNN
-F 1 "4.7k" V 6300 2600 50  0000 C CNN
-F 2 "" V 6230 2600 30  0000 C CNN
-F 3 "" H 6300 2600 30  0000 C CNN
-	1    6300 2600
-	1    0    0    -1
-$EndComp
-$Comp
-L R R4
-U 1 1 554CCD26
-P 6300 4400
-F 0 "R4" V 6380 4400 50  0000 C CNN
-F 1 "1k" V 6300 4400 50  0000 C CNN
-F 2 "" V 6230 4400 30  0000 C CNN
-F 3 "" H 6300 4400 30  0000 C CNN
-	1    6300 4400
-	1    0    0    -1
-$EndComp
-$Comp
-L R R1
-U 1 1 554CCD86
-P 4100 3500
-F 0 "R1" V 4180 3500 50  0000 C CNN
-F 1 "10k" V 4100 3500 50  0000 C CNN
-F 2 "" V 4030 3500 30  0000 C CNN
-F 3 "" H 4100 3500 30  0000 C CNN
-	1    4100 3500
-	0    1    1    0
-$EndComp
-$Comp
 L C C1
 U 1 1 554CCDF0
@@
 $EndComp
 $Comp
-L R R2
-U 1 1 554CCF0B
-P 5150 4300
-F 0 "R2" V 5230 4300 50  0000 C CNN
-F 1 "1Meg" V 5150 4300 50  0000 C CNN
-F 2 "" V 5080 4300 30  0000 C CNN
-F 3 "" H 5150 4300 30  0000 C CNN
-	1    5150 4300
-	-1   0    0    1
-$EndComp
-$Comp
 L C C2
 U 1 1 554CCF4F
@@
 $EndComp
 $Comp
-L R R5
-U 1 1 554CD260
-P 8600 3750
-F 0 "R5" V 8680 3750 50  0000 C CNN
-F 1 "2.2k" V 8600 3750 50  0000 C CNN
-F 2 "" V 8530 3750 30  0000 C CNN
-F 3 "" H 8600 3750 30  0000 C CNN
-	1    8600 3750
-	1    0    0    -1
-$EndComp
-$Comp
 L GND #PWR01
 U 1 1 554CD6B0
@@
 $EndComp
 Wire Wire Line
-	6300 3300 6300 2750
-Wire Wire Line
-	6300 4250 6300 3700
+	6300 2750 6300 3300
+Wire Wire Line
+	6300 3700 6300 4250
 Wire Wire Line
 	4800 3500 6000 3500
@@
 	3550 4750 3550 4800
 Connection ~ 5150 4800
-$Comp
-L vplot8_1 U1
-U 1 1 554CE506
-P 3550 3100
-F 0 "U1" H 3400 3200 50  0000 C CNN
-F 1 "vplot8_1" H 3700 3200 50  0000 C CNN
-F 2 "" H 3550 3100 60  0000 C CNN
-F 3 "" H 3550 3100 60  0000 C CNN
-	1    3550 3100
-	1    0    0    -1
-$EndComp
-$Comp
-L vplot8_1 U2
-U 2 1 554CE5B6
-P 8500 2750
-F 0 "U2" H 8350 2850 50  0000 C CNN
-F 1 "vplot8_1" H 8650 2850 50  0000 C CNN
-F 2 "" H 8500 2750 60  0000 C CNN
-F 3 "" H 8500 2750 60  0000 C CNN
-	2    8500 2750
-	1    0    0    -1
-$EndComp
 Wire Wire Line
 	8500 3050 8500 3100
@@
 	1    0    0    -1
 $EndComp
+$Comp
+L R R3
+U 1 1 55D44D80
+P 6250 2550
+F 0 "R3" H 6300 2680 50  0000 C CNN
+F 1 "4.7k" H 6300 2600 50  0000 C CNN
+F 2 "" H 6300 2530 30  0000 C CNN
+F 3 "" V 6300 2600 30  0000 C CNN
+	1    6250 2550
+	0    1    1    0
+$EndComp
+$Comp
+L R R1
+U 1 1 55D44DE3
+P 4050 3550
+F 0 "R1" H 4100 3680 50  0000 C CNN
+F 1 "10k" H 4100 3600 50  0000 C CNN
+F 2 "" H 4100 3530 30  0000 C CNN
+F 3 "" V 4100 3600 30  0000 C CNN
+	1    4050 3550
+	1    0    0    -1
+$EndComp
+$Comp
+L R R2
+U 1 1 55D44EE5
+P 5200 4350
+F 0 "R2" H 5250 4480 50  0000 C CNN
+F 1 "1Meg" H 5250 4400 50  0000 C CNN
+F 2 "" H 5250 4330 30  0000 C CNN
+F 3 "" V 5250 4400 30  0000 C CNN
+	1    5200 4350
+	0    -1   -1   0
+$EndComp
+$Comp
+L R R4
+U 1 1 55D44F9D
+P 6350 4450
+F 0 "R4" H 6400 4580 50  0000 C CNN
+F 1 "1k" H 6400 4500 50  0000 C CNN
+F 2 "" H 6400 4430 30  0000 C CNN
+F 3 "" V 6400 4500 30  0000 C CNN
+	1    6350 4450
+	0    -1   -1   0
+$EndComp
+$Comp
+L R R5
+U 1 1 55D45045
+P 8650 3800
+F 0 "R5" H 8700 3930 50  0000 C CNN
+F 1 "2.2k" H 8700 3850 50  0000 C CNN
+F 2 "" H 8700 3780 30  0000 C CNN
+F 3 "" V 8700 3850 30  0000 C CNN
+	1    8650 3800
+	0    -1   -1   0
+$EndComp
+Text GLabel 8500 3050 1    60   Input ~ 0
+Out
+Text GLabel 3550 3400 1    60   Input ~ 0
+in
 $EndSCHEMATC

Commit message: Remove unwanted example
Parts:
- removed C2: 5p, symbol C
- removed C3: 4p, symbol C
- removed C4: 2p, symbol C
- removed C5: 0.5p, symbol C
- removed C7: 5u, symbol C
- removed C8: 6p, symbol C
- removed R1: 10k, symbol R
- removed R5: 2.2k, symbol R
- added U1: plot_v1, symbol plot_v1
- added U2: plot_phase, symbol plot_phase
- added U3: plot_log, symbol plot_log
- added U4: plot_db, symbol plot_db
- C1: value 0.01u -> 1u
- C6: value 2u -> 0.1u
- R3: value 4.7k -> 3k
- R4: value 1k -> 470
- v2: value dc -> DC; symbol dc -> DC
Connections:
- net labels added: out
- net labels removed: Out
- wire segments 34 -> 21
Changed lines of the file:
@@
 EESchema Schematic File Version 2
+LIBS:FrequencyResponse_JFET-rescue
 LIBS:eSim_Analog
 LIBS:eSim_Devices
@@
 LIBS:eSim_Hybrid
 LIBS:eSim_Miscellaneous
+LIBS:eSim_Plot
+LIBS:eSim_Power
 LIBS:eSim_Sources
 LIBS:eSim_Subckt
@@
 P 4650 3500
 F 0 "C1" H 4675 3600 50  0000 L CNN
-F 1 "0.01u" H 4675 3400 50  0000 L CNN
+F 1 "1u" H 4675 3400 50  0000 L CNN
 F 2 "" H 4688 3350 30  0000 C CNN
 F 3 "" H 4650 3500 60  0000 C CNN
@@
 $EndComp
 $Comp
-L C C2
-U 1 1 554CCF4F
-P 5450 4300
-F 0 "C2" H 5475 4400 50  0000 L CNN
-F 1 "5p" H 5475 4200 50  0000 L CNN
-F 2 "" H 5488 4150 30  0000 C CNN
-F 3 "" H 5450 4300 60  0000 C CNN
-	1    5450 4300
-	-1   0    0    1
-$EndComp
-$Comp
-L C C3
-U 1 1 554CCFBE
-P 5950 3900
-F 0 "C3" H 5975 4000 50  0000 L CNN
-F 1 "4p" H 5975 3800 50  0000 L CNN
-F 2 "" H 5988 3750 30  0000 C CNN
-F 3 "" H 5950 3900 60  0000 C CNN
-	1    5950 3900
-	0    -1   -1   0
-$EndComp
-$Comp
-L C C4
-U 1 1 554CCFFC
-P 6000 3100
-F 0 "C4" H 6025 3200 50  0000 L CNN
-F 1 "2p" H 6025 3000 50  0000 L CNN
-F 2 "" H 6038 2950 30  0000 C CNN
-F 3 "" H 6000 3100 60  0000 C CNN
-	1    6000 3100
-	0    -1   -1   0
-$EndComp
-$Comp
-L C C5
-U 1 1 554CD040
-P 6750 3550
-F 0 "C5" H 6775 3650 50  0000 L CNN
-F 1 "0.5p" H 6775 3450 50  0000 L CNN
-F 2 "" H 6788 3400 30  0000 C CNN
-F 3 "" H 6750 3550 60  0000 C CNN
-	1    6750 3550
-	1    0    0    -1
-$EndComp
-$Comp
 L C C6
 U 1 1 554CD166
 P 6750 4350
 F 0 "C6" H 6775 4450 50  0000 L CNN
-F 1 "2u" H 6775 4250 50  0000 L CNN
+F 1 "0.1u" H 6775 4250 50  0000 L CNN
 F 2 "" H 6788 4200 30  0000 C CNN
 F 3 "" H 6750 4350 60  0000 C CNN
 	1    6750 4350
-	1    0    0    -1
-$EndComp
-$Comp
-L C C7
-U 1 1 554CD1B0
-P 7350 3100
-F 0 "C7" H 7375 3200 50  0000 L CNN
-F 1 "5u" H 7375 3000 50  0000 L CNN
-F 2 "" H 7388 2950 30  0000 C CNN
-F 3 "" H 7350 3100 60  0000 C CNN
-	1    7350 3100
-	0    -1   -1   0
-$EndComp
-$Comp
-L C C8
-U 1 1 554CD20C
-P 8200 3700
-F 0 "C8" H 8225 3800 50  0000 L CNN
-F 1 "6p" H 8225 3600 50  0000 L CNN
-F 2 "" H 8238 3550 30  0000 C CNN
-F 3 "" H 8200 3700 60  0000 C CNN
-	1    8200 3700
 	1    0    0    -1
 $EndComp
@@
 $EndComp
 $Comp
-L dc v2
+L DC v2
 U 1 1 554CD920
-P 6300 1800
-F 0 "v2" H 6100 1900 60  0000 C CNN
-F 1 "dc" H 6100 1750 60  0000 C CNN
-F 2 "R1" H 6000 1800 60  0000 C CNN
-F 3 "" H 6300 1800 60  0000 C CNN
-	1    6300 1800
-	-1   0    0    1
-$EndComp
-$Comp
-L GND #PWR02
-U 1 1 554CDAE1
-P 6750 1350
-F 0 "#PWR02" H 6750 1100 50  0001 C CNN
-F 1 "GND" H 6750 1200 50  0000 C CNN
-F 2 "" H 6750 1350 60  0000 C CNN
-F 3 "" H 6750 1350 60  0000 C CNN
-	1    6750 1350
+P 8600 3650
+F 0 "v2" H 8400 3750 60  0000 C CNN
+F 1 "DC" H 8400 3600 60  0000 C CNN
+F 2 "R1" H 8300 3650 60  0000 C CNN
+F 3 "" H 8600 3650 60  0000 C CNN
+	1    8600 3650
 	1    0    0    -1
 $EndComp
@@
 Wire Wire Line
 	4800 3500 6000 3500
-Wire Wire Line
-	5450 4150 5450 3500
-Connection ~ 5450 3500
 Wire Wire Line
 	5150 4150 5150 3500
 Connection ~ 5150 3500
-Wire Wire Line
-	5650 3900 5800 3900
-Wire Wire Line
-	5650 3100 5650 3900
-Connection ~ 5650 3500
-Wire Wire Line
-	6100 3900 6750 3900
-Connection ~ 6300 3900
-Wire Wire Line
-	6750 3900 6750 3700
-Wire Wire Line
-	6150 3100 7200 3100
 Connection ~ 6300 3100
-Wire Wire Line
-	6750 3100 6750 3400
-Wire Wire Line
-	5850 3100 5650 3100
-Connection ~ 6750 3100
-Wire Wire Line
-	7500 3100 8600 3100
-Wire Wire Line
-	8600 3100 8600 3600
-Wire Wire Line
-	8200 3550 8200 3100
-Connection ~ 8200 3100
 Wire Wire Line
 	6750 4200 6750 4100
@@
 	6300 4550 6300 4850
 Wire Wire Line
-	4250 3500 4500 3500
+	3550 3500 4500 3500
 Wire Wire Line
 	5150 4450 5150 4800
@@
 Connection ~ 6300 4800
 Wire Wire Line
-	8600 4800 8600 3900
-Wire Wire Line
-	8200 3850 8200 4800
-Connection ~ 8200 4800
-Wire Wire Line
 	6750 4500 6750 4800
 Connection ~ 6750 4800
 Wire Wire Line
-	5450 4450 5450 4800
-Connection ~ 5450 4800
-Wire Wire Line
 	6300 2250 6300 2450
-Wire Wire Line
-	6300 1350 6300 1250
-Wire Wire Line
-	6300 1250 6750 1250
-Wire Wire Line
-	6750 1250 6750 1350
-Wire Wire Line
-	3950 3500 3550 3500
-Wire Wire Line
-	3550 3400 3550 3850
 Wire Wire Line
 	3550 4750 3550 4800
 Connection ~ 5150 4800
-Wire Wire Line
-	8500 3050 8500 3100
-Connection ~ 8500 3100
-Connection ~ 3550 3500
-$Comp
-L PWR_FLAG #FLG03
-U 1 1 554CEAE9
-P 6500 1200
-F 0 "#FLG03" H 6500 1295 50  0001 C CNN
-F 1 "PWR_FLAG" H 6500 1380 50  0000 C CNN
-F 2 "" H 6500 1200 60  0000 C CNN
-F 3 "" H 6500 1200 60  0000 C CNN
-	1    6500 1200
-	1    0    0    -1
-$EndComp
-Wire Wire Line
-	6500 1200 6500 1250
-Connection ~ 6500 1250
-$Comp
-L AC v1
-U 1 1 554CED04
-P 3550 4300
-F 0 "v1" H 3350 4400 60  0000 C CNN
-F 1 "AC" H 3350 4250 60  0000 C CNN
-F 2 "R1" H 3250 4300 60  0000 C CNN
-F 3 "" H 3550 4300 60  0000 C CNN
-	1    3550 4300
-	1    0    0    -1
-$EndComp
 $Comp
 L NJF J1
@@
 P 6250 2550
 F 0 "R3" H 6300 2680 50  0000 C CNN
-F 1 "4.7k" H 6300 2600 50  0000 C CNN
+F 1 "3k" H 6300 2600 50  0000 C CNN
 F 2 "" H 6300 2530 30  0000 C CNN
 F 3 "" V 6300 2600 30  0000 C CNN
 	1    6250 2550
 	0    1    1    0
-$EndComp
-$Comp
-L R R1
-U 1 1 55D44DE3
-P 4050 3550
-F 0 "R1" H 4100 3680 50  0000 C CNN
-F 1 "10k" H 4100 3600 50  0000 C CNN
-F 2 "" H 4100 3530 30  0000 C CNN
-F 3 "" V 4100 3600 30  0000 C CNN
-	1    4050 3550
-	1    0    0    -1
 $EndComp
 $Comp
@@
 P 6350 4450
 F 0 "R4" H 6400 4580 50  0000 C CNN
-F 1 "1k" H 6400 4500 50  0000 C CNN
+F 1 "470" H 6400 4500 50  0000 C CNN
 F 2 "" H 6400 4430 30  0000 C CNN
 F 3 "" V 6400 4500 30  0000 C CNN
@@
 	0    -1   -1   0
 $EndComp
-$Comp
-L R R5
-U 1 1 55D45045
-P 8650 3800
-F 0 "R5" H 8700 3930 50  0000 C CNN
-F 1 "2.2k" H 8700 3850 50  0000 C CNN
-F 2 "" H 8700 3780 30  0000 C CNN
-F 3 "" V 8700 3850 30  0000 C CNN
-	1    8650 3800
-	0    -1   -1   0
-$EndComp
-Text GLabel 8500 3050 1    60   Input ~ 0
-Out
-Text GLabel 3550 3400 1    60   Input ~ 0
+Text GLabel 3350 3350 0    60   Input ~ 0
 in
+Wire Wire Line
+	6300 2250 8600 2250
+Wire Wire Line
+	8600 2250 8600 3200
+Wire Wire Line
+	8600 4800 8600 4100
+Text GLabel 7300 3100 2    60   Input ~ 0
+out
+Wire Wire Line
+	6300 3100 7300 3100
+$Comp
+L plot_v1 U1
+U 1 1 56D858F3
+P 3550 3400
+F 0 "U1" H 3550 3900 60  0000 C CNN
+F 1 "plot_v1" H 3750 3750 60  0000 C CNN
+F 2 "" H 3550 3400 60  0000 C CNN
+F 3 "" H 3550 3400 60  0000 C CNN
+	1    3550 3400
+	1    0    0    -1
+$EndComp
+Wire Wire Line
+	6600 3050 6600 3250
+Connection ~ 6600 3100
+Wire Wire Line
+	3550 3200 3550 3850
+Connection ~ 3550 3500
+Wire Wire Line
+	3350 3350 3550 3350
+Connection ~ 3550 3350
+$Comp
+L AC v1
+U 1 1 56D85DA9
+P 3550 4300
+F 0 "v1" H 3350 4400 60  0000 C CNN
+F 1 "AC" H 3350 4250 60  0000 C CNN
+F 2 "R1" H 3250 4300 60  0000 C CNN
+F 3 "" H 3550 4300 60  0000 C CNN
+	1    3550 4300
+	1    0    0    -1
+$EndComp
+$Comp
+L plot_log U3
+U 1 1 56D85E87
+P 6600 3250
+F 0 "U3" H 6600 3750 60  0000 C CNN
+F 1 "plot_log" H 6800 3600 60  0000 C CNN
+F 2 "" H 6600 3250 60  0000 C CNN
+F 3 "" H 6600 3250 60  0000 C CNN
+	1    6600 3250
+	1    0    0    -1
+$EndComp
+$Comp
+L plot_phase U2
+U 1 1 56D85EE2
+P 6600 3050
+F 0 "U2" H 6600 3550 60  0000 C CNN
+F 1 "plot_phase" H 6850 3400 60  0000 C CNN
+F 2 "" H 6600 3050 60  0000 C CNN
+F 3 "" H 6600 3050 60  0000 C CNN
+	1    6600 3050
+	1    0    0    1
+$EndComp
+$Comp
+L plot_db U4
+U 1 1 56D86013
+P 7100 3250
+F 0 "U4" H 7100 3750 60  0000 C CNN
+F 1 "plot_db" H 7300 3600 60  0000 C CNN
+F 2 "" H 7100 3250 60  0000 C CNN
+F 3 "" H 7100 3250 60  0000 C CNN
+	1    7100 3250
+	1    0    0    -1
+$EndComp
+Wire Wire Line
+	7100 3050 7100 3100
+Connection ~ 7100 3100
 $EndSCHEMATC

Commit message: common code for Win and Linux, merged py2 changes
Parts:
- removed J1: NJF, symbol NJF
- added J1: eSim_NJF, symbol eSim_NJF
- R2, R3, R4: symbol R -> R-RESCUE-FrequencyResponse_JFET
- v2: symbol DC -> DC-RESCUE-FrequencyResponse_JFET
Connections:
- net out: now also J1.1 (D)
- net at C1.1, R2.2: now also J1.2 (G)
- net at C6.1, R4.2: now also J1.3 (S)
Changed lines of the file:
@@
 $EndComp
 $Comp
-L DC v2
+L DC-RESCUE-FrequencyResponse_JFET v2
 U 1 1 554CD920
 P 8600 3650
@@
 Connection ~ 5150 4800
 $Comp
-L NJF J1
-U 1 1 557065CE
-P 6200 3500
-F 0 "J1" H 6100 3550 50  0000 R CNN
-F 1 "NJF" H 6150 3650 50  0000 R CNN
-F 2 "" H 6400 3600 29  0000 C CNN
-F 3 "" H 6200 3500 60  0000 C CNN
-	1    6200 3500
-	1    0    0    -1
-$EndComp
-$Comp
-L R R3
+L R-RESCUE-FrequencyResponse_JFET R3
 U 1 1 55D44D80
 P 6250 2550
@@
 $EndComp
 $Comp
-L R R2
+L R-RESCUE-FrequencyResponse_JFET R2
 U 1 1 55D44EE5
 P 5200 4350
@@
 $EndComp
 $Comp
-L R R4
+L R-RESCUE-FrequencyResponse_JFET R4
 U 1 1 55D44F9D
 P 6350 4450
@@
 	7100 3050 7100 3100
 Connection ~ 7100 3100
+$Comp
+L eSim_NJF J1
+U 1 1 5D676245
+P 6200 3500
+F 0 "J1" H 6100 3550 50  0000 R CNN
+F 1 "eSim_NJF" H 6150 3650 50  0000 R CNN
+F 2 "" H 6400 3600 29  0000 C CNN
+F 3 "" H 6200 3500 60  0000 C CNN
+	1    6200 3500
+	1    0    0    -1
+$EndComp
+$Comp
+L PWR_FLAG #FLG02
+U 1 1 5D67639B
+P 6550 4600
+F 0 "#FLG02" H 6550 4675 50  0001 C CNN
+F 1 "PWR_FLAG" H 6550 4750 50  0000 C CNN
+F 2 "" H 6550 4600 50  0001 C CNN
+F 3 "" H 6550 4600 50  0001 C CNN
+	1    6550 4600
+	1    0    0    -1
+$EndComp
+Wire Wire Line
+	6550 4600 6550 4800
+Connection ~ 6550 4800
 $EndSCHEMATC
