File: Examples/Fullwavebridgerectifier/Fullwavebridgerectifier.sch (KiCad schematic (older format))
At the start: 8 parts, among them U1 plot_v2, U2 plot_v1

Commit message: common code for Win and Linux, merged py2 changes
Parts:
- D1, D2, D3, D4: symbol D -> D-RESCUE-Fullwavebridgerectifier
- R1: symbol R -> R-RESCUE-Fullwavebridgerectifier
Changed lines of the file:
@@
 EESchema Schematic File Version 2
+LIBS:Fullwavebridgerectifier-rescue
 LIBS:eSim_Analog
 LIBS:eSim_Devices
@@
 $EndComp
 $Comp
-L D D1
+L D-RESCUE-Fullwavebridgerectifier D1
 U 1 1 56A85EED
 P 4200 2900
@@
 $EndComp
 $Comp
-L D D3
+L D-RESCUE-Fullwavebridgerectifier D3
 U 1 1 56A85F6E
 P 5000 2900
@@
 $EndComp
 $Comp
-L D D2
+L D-RESCUE-Fullwavebridgerectifier D2
 U 1 1 56A85FBD
 P 4200 4250
@@
 $EndComp
 $Comp
-L D D4
+L D-RESCUE-Fullwavebridgerectifier D4
 U 1 1 56A8602F
 P 5000 4250
@@
 $EndComp
 $Comp
-L R R1
+L R-RESCUE-Fullwavebridgerectifier R1
 U 1 1 56A860D7
 P 6050 3400
