File: Examples/Parallel_Resonance/Parallel_Resonance.sch (KiCad schematic (older format))
At the start: 7 parts, among them U1 plot_v1, U3 plot_v1

Commit message: common code for Win and Linux, merged py2 changes
Parts:
- L1: symbol L -> L-RESCUE-Parallel_Resonance
- R1, R2: symbol R -> R-RESCUE-Parallel_Resonance
Changed lines of the file:
@@
 EESchema Schematic File Version 2
+LIBS:Parallel_Resonance-rescue
 LIBS:eSim_Analog
 LIBS:eSim_Devices
@@
 $EndDescr
 $Comp
-L R R1
+L R-RESCUE-Parallel_Resonance R1
 U 1 1 56C172A1
 P 5100 3150
@@
 $EndComp
 $Comp
-L L L1
+L L-RESCUE-Parallel_Resonance L1
 U 1 1 56C172D6
 P 5850 1250
@@
 Connection ~ 5900 3850
 $Comp
-L R R2
+L R-RESCUE-Parallel_Resonance R2
 U 1 1 56C1A863
 P 4600 2600
