File: Examples/RC/RC.sch (KiCad schematic (older format))
At the start: 5 parts, among them U1 plot_v1, U2 plot_v1

Commit message: common code for Win and Linux, merged py2 changes
Parts:
- R1: symbol R -> R-RESCUE-RC
Changed lines of the file:
@@
 EESchema Schematic File Version 2
+LIBS:RC-rescue
 LIBS:eSim_Analog
 LIBS:eSim_Devices
@@
 $EndDescr
 $Comp
-L R R1
+L R-RESCUE-RC R1
 U 1 1 56B86791
 P 5750 3050
