File: src/SubcircuitLibrary/74153/4_and.sch (KiCad schematic (older format))
At the start: 3 parts, among them U1 PORT, U2 d_and, X1 3_and

Commit message: common code for Win and Linux, merged py2 changes
Parts:
- X1: symbol 3_and-RESCUE-4_and -> 3_and
Other:
- note removed: "in1"
- note removed: "in2"
- note removed: "in3"
- note removed: "in4"
- note removed: "out"
Changed lines of the file:
@@
 EESchema Schematic File Version 2
-LIBS:4_and-rescue
 LIBS:texas
 LIBS:intel
@@
 LIBS:eSim_Subckt
 LIBS:eSim_User
-LIBS:4_and-cache
 EELAYER 25 0
 EELAYER END
@@
 $EndDescr
 $Comp
-L 3_and-RESCUE-4_and X1
+L 3_and X1
 U 1 1 5C9A2915
 P 3700 3500
@@
 	-1   0    0    1
 $EndComp
-Text Notes 3450 2650 0    60   ~ 12
-in1
-Text Notes 3450 2950 0    60   ~ 12
-in2
-Text Notes 3500 3300 0    60   ~ 12
-in3
-Text Notes 3500 3550 0    60   ~ 12
-in4
-Text Notes 6150 3350 0    60   ~ 12
-out
 $EndSCHEMATC
