File: src/SubcircuitLibrary/74157/74157.sch (KiCad schematic (older format))
At the start: 15 parts, among them U1 PORT, U2 d_inverter, U20 d_or, U21 d_or, U22 d_or, U23 d_or, U3 d_inverter, X1 3_and, X2 3_and, X3 3_and, X4 3_and, X5 3_and, X6 3_and, X7 3_and, X8 3_and

Commit message: common code for Win and Linux, merged py2 changes
Parts:
- removed unit 8 of U1
- removed unit 16 of U1
- X1, X2, X3, X4, X5, X6, X7, X8: symbol 3_and-RESCUE-74157 -> 3_and
Connections:
- no-connect marks 2 -> 0
Other:
- moved on the sheet: U1E, U1F
