File: src/SubcircuitLibrary/7485/7485.sch (KiCad schematic (older format))
At the start: 32 parts, among them U1 PORT, U10 d_and, U11 d_and, U12 d_and, U13 d_and, U14 d_nor, U15 d_nor, U16 d_nor, U17 d_nor, U18 d_and, U19 d_and, U2 d_nand, U3 d_nand, U4 d_nand, U5 d_nand, U6 d_and, U7 d_and, U8 d_and, U9 d_and, X1 5_nor, X10 5_and, X11 5_and, X12 5_nor, X13 5_and, X2 3_and, X3 4_and, X4 5_and, X5 5_and, X6 5_and, X7 3_and, X8 4_and, X9 5_and

Commit message: common code for Win and Linux, merged py2 changes
Parts:
- removed unit 8 of U1
- removed unit 16 of U1
- removed X1, X12: 5_nor, symbol 5_nor
- removed X2, X7: 3_and, symbol 3_and
- removed X8: 4_and, symbol 4_and
- added X1, X2: c_gate, symbol c_gate
- added X12, X8: 3_and, symbol 3_and
- added X7: 4_and, symbol 4_and
Connections:
- wire segments 182 -> 242
- no-connect marks 3 -> 0
