File: src/SubcircuitLibrary/ujt/ujt.sch (KiCad schematic (older format))
At the start: 8 parts, among them U1 PORT

Commit message: common code for Win and Linux, merged py2 changes
Parts:
- R1: value 38.15 -> 38.15k
Connections:
- net labels added: 0
- net labels removed: GND
- wire segments 19 -> 21
Other:
- moved on the sheet: D1, R3, U1A
Changed lines of the file:
@@
 L eSim_R R3
 U 1 1 5CF5F733
-P 7400 2850
-F 0 "R3" H 7450 2980 50  0000 C CNN
-F 1 "1000k" H 7450 2900 50  0000 C CNN
-F 2 "" H 7450 2830 30  0000 C CNN
-F 3 "" V 7450 2900 30  0000 C CNN
-	1    7400 2850
+P 6650 3400
+F 0 "R3" H 6700 3530 50  0000 C CNN
+F 1 "1000k" H 6700 3450 50  0000 C CNN
+F 2 "" H 6700 3380 30  0000 C CNN
+F 3 "" V 6700 3450 30  0000 C CNN
+	1    6650 3400
 	0    1    -1   0
+$EndComp
+$Comp
+L CCVS H1
+U 1 1 5CF5F77B
+P 6150 3350
+F 0 "H1" H 6150 3500 50  0000 C CNN
+F 1 "1k" H 5950 3300 50  0000 C CNN
+F 2 "" H 6150 3350 60  0000 C CNN
+F 3 "" H 6150 3350 60  0000 C CNN
+	1    6150 3350
+	0    1    1    0
 $EndComp
 $Comp
@@
 P 4300 4850
 F 0 "R1" H 4350 4980 50  0000 C CNN
-F 1 "38.15" H 4350 4900 50  0000 C CNN
+F 1 "38.15k" H 4350 4900 50  0000 C CNN
 F 2 "" H 4350 4830 30  0000 C CNN
 F 3 "" V 4350 4900 30  0000 C CNN
@@
 L PORT U1
 U 1 1 5CF689AD
-P 5950 1200
-F 0 "U1" H 6000 1300 30  0000 C CNN
-F 1 "PORT" H 5950 1200 30  0000 C CNN
-F 2 "" H 5950 1200 60  0000 C CNN
-F 3 "" H 5950 1200 60  0000 C CNN
-	1    5950 1200
+P 5950 2200
+F 0 "U1" H 6000 2300 30  0000 C CNN
+F 1 "PORT" H 5950 2200 30  0000 C CNN
+F 2 "" H 5950 2200 60  0000 C CNN
+F 3 "" H 5950 2200 60  0000 C CNN
+	1    5950 2200
 	0    1    1    0
 $EndComp
@@
 	0    1    1    0
 $EndComp
+Text Label 5600 4100 0    60   ~ 0
+5
+Text Label 5950 3150 0    60   ~ 0
+4
+Text Label 5950 2600 0    60   ~ 0
+1
+Text Label 6450 3050 0    60   ~ 0
+6
+Text Label 6450 3650 0    60   ~ 0
+0
 $Comp
 L NLDS B1
@@
 	1    0    0    -1
 $EndComp
+Text Label 5350 5250 0    60   ~ 0
+7
+Text Label 4600 3450 0    60   ~ 0
+3
+Text Label 4250 4500 0    60   ~ 0
+2
 $Comp
 L eSim_Diode D1
 U 1 1 5CFF8BB7
-P 5950 1850
-F 0 "D1" H 5950 1950 50  0000 C CNN
-F 1 "eSim_Diode" H 5950 1750 50  0000 C CNN
-F 2 "" H 5950 1850 60  0000 C CNN
-F 3 "" H 5950 1850 60  0000 C CNN
-	1    5950 1850
+P 5950 2850
+F 0 "D1" H 5950 2950 50  0000 C CNN
+F 1 "eSim_Diode" H 5950 2750 50  0000 C CNN
+F 2 "" H 5950 2850 60  0000 C CNN
+F 3 "" H 5950 2850 60  0000 C CNN
+	1    5950 2850
 	0    1    1    0
 $EndComp
 Wire Wire Line
-	6950 2500 7450 2500
+	6200 3050 6700 3050
 Wire Wire Line
-	7450 2500 7450 2650
+	6700 3050 6700 3200
 Wire Wire Line
-	6950 3100 7450 3100
+	6200 3650 6300 3650
 Wire Wire Line
-	5950 1450 5950 1700
+	6300 3650 6700 3650
 Wire Wire Line
-	5950 2000 5950 2750
+	5950 2450 5950 2700
 Wire Wire Line
-	5950 2850 5950 4450
+	5950 3000 5950 3300
+Wire Wire Line
+	5950 3400 5950 3850
+Wire Wire Line
+	5950 3850 5950 4100
+Wire Wire Line
+	5950 4100 5950 4450
 Wire Wire Line
 	5150 4100 5150 4550
 Wire Wire Line
-	4600 4100 5950 4100
+	4600 4100 5150 4100
+Wire Wire Line
+	5150 4100 5950 4100
+Connection ~ 5950 4100
 Wire Wire Line
 	5150 4850 5150 5250
 Wire Wire Line
-	4250 5250 5950 5250
+	4250 5250 5150 5250
+Wire Wire Line
+	5150 5250 5950 5250
 Wire Wire Line
 	4250 5250 4250 4950
@@
 Connection ~ 5150 5250
 Wire Wire Line
-	7450 3100 7450 2950
-Connection ~ 5950 4100
-$Comp
-L CCVS H1
-U 1 1 5D04A7ED
-P 6900 2800
-F 0 "H1" H 6900 2950 50  0000 C CNN
-F 1 "1k" H 6700 2750 50  0000 C CNN
-F 2 "" H 6900 2800 60  0000 C CNN
-F 3 "" H 6900 2800 60  0000 C CNN
-	1    6900 2800
-	0    1    1    0
-$EndComp
-$Comp
-L GND #PWR01
-U 1 1 5D04C560
-P 7150 3150
-F 0 "#PWR01" H 7150 2900 50  0001 C CNN
-F 1 "GND" H 7150 3000 50  0000 C CNN
-F 2 "" H 7150 3150 50  0001 C CNN
-F 3 "" H 7150 3150 50  0001 C CNN
-	1    7150 3150
-	1    0    0    -1
-$EndComp
-Wire Wire Line
-	7150 3150 7150 3100
-Connection ~ 7150 3100
-Wire Wire Line
-	5950 2750 6700 2750
-Wire Wire Line
-	6700 2850 5950 2850
-Text GLabel 5950 1550 0    60   Input ~ 0
-1
-Text GLabel 5950 2200 0    60   Input ~ 0
-4
-Text GLabel 5950 3500 0    60   Input ~ 0
-5
-Text GLabel 5700 5250 3    60   Input ~ 0
-7
-Text GLabel 4250 4550 0    60   Input ~ 0
-2
-Text GLabel 4600 3350 0    60   Input ~ 0
-3
-Text GLabel 7200 2500 1    60   Input ~ 0
-6
+	6700 3650 6700 3500
 $EndSCHEMATC
