File: Examples/FullAdder/FullAdder.sch (KiCad schematic (older format))
At the start: 13 parts, among them U1 plot_v1, U2 plot_v1, U3 plot_v1, U4 plot_v1, U5 plot_v1, U6 adc_bridge_3, U7 dac_bridge_2, X1 full_adder

Commit message: part2/3 - .pro cleanup
Parts:
- v1, v2, v3: symbol DC -> DC-RESCUE-FullAdder
Changed lines of the file:
@@
 EESchema Schematic File Version 2
+LIBS:FullAdder-rescue
 LIBS:eSim_Analog
 LIBS:eSim_Devices
@@
 LIBS:contrib
 LIBS:power
-LIBS:device
 LIBS:transistors
 LIBS:conn
-LIBS:linear
 LIBS:regul
 LIBS:74xx
 LIBS:cmos4000
+LIBS:FullAdder-cache
 EELAYER 25 0
 EELAYER END
@@
 $EndComp
 $Comp
-L DC v1
+L DC-RESCUE-FullAdder v1
 U 1 1 56D58CB2
 P 1300 3550
@@
 $EndComp
 $Comp
-L DC v2
+L DC-RESCUE-FullAdder v2
 U 1 1 56D58D3D
 P 1950 3950
@@
 $EndComp
 $Comp
-L DC v3
+L DC-RESCUE-FullAdder v3
 U 1 1 56D58D84
 P 2700 4350
