File: Examples/Integrator/Integrator.sch (KiCad schematic (older format))
At the start: 9 parts, among them U1 plot_v1, U2 plot_v1, X1 UA741

Commit message: common code for Win and Linux, merged py2 changes
Parts:
- R1, R2, R3, R4: symbol R -> R-RESCUE-Integrator
Changed lines of the file:
@@
 EESchema Schematic File Version 2
+LIBS:Integrator-rescue
 LIBS:eSim_Analog
 LIBS:eSim_Devices
@@
 LIBS:74xx
 LIBS:cmos4000
-LIBS:Integrator-cache
 EELAYER 25 0
 EELAYER END
@@
 $EndComp
 $Comp
-L R R1
+L R-RESCUE-Integrator R1
 U 1 1 56A9B635
 P 5100 3150
@@
 $EndComp
 $Comp
-L R R2
+L R-RESCUE-Integrator R2
 U 1 1 56A9B674
 P 5400 3400
@@
 $EndComp
 $Comp
-L R R3
+L R-RESCUE-Integrator R3
 U 1 1 56A9B6AE
 P 6850 3300
@@
 	6650 2350 6650 3200
 $Comp
-L R R4
+L R-RESCUE-Integrator R4
 U 1 1 56B2EBCB
 P 6050 2400

Commit message: part2/3 - .pro cleanup
Parts:
- removed C1: 100n, symbol C
- removed R1: 10k, symbol R-RESCUE-Integrator
- removed R2, R3: 1k, symbol R-RESCUE-Integrator
- removed R4: 100k, symbol R-RESCUE-Integrator
- added C1: 100n, symbol capacitor
- added R1: 10k, symbol resistor
- added R2, R4: 1k, symbol resistor
- added R3: 100k, symbol resistor
Other:
- note added: "100k\n"
- note added: "100n"
- note added: "10k"
- note added: "1k"
- note added: "1k\n"
Changed lines of the file:
@@
 EESchema Schematic File Version 2
-LIBS:Integrator-rescue
 LIBS:eSim_Analog
 LIBS:eSim_Devices
@@
 LIBS:contrib
 LIBS:power
-LIBS:device
 LIBS:transistors
 LIBS:conn
-LIBS:linear
 LIBS:regul
 LIBS:74xx
@@
 	1    0    0    1
 $EndComp
-$Comp
-L R-RESCUE-Integrator R1
-U 1 1 56A9B635
-P 5100 3150
-F 0 "R1" H 5150 3280 50  0000 C CNN
-F 1 "10k" H 5150 3200 50  0000 C CNN
-F 2 "" H 5150 3130 30  0000 C CNN
-F 3 "" V 5150 3200 30  0000 C CNN
-	1    5100 3150
-	1    0    0    -1
-$EndComp
-$Comp
-L R-RESCUE-Integrator R2
-U 1 1 56A9B674
-P 5400 3400
-F 0 "R2" H 5450 3530 50  0000 C CNN
-F 1 "1k" H 5450 3450 50  0000 C CNN
-F 2 "" H 5450 3380 30  0000 C CNN
-F 3 "" V 5450 3450 30  0000 C CNN
-	1    5400 3400
-	0    1    1    0
-$EndComp
-$Comp
-L R-RESCUE-Integrator R3
-U 1 1 56A9B6AE
-P 6850 3300
-F 0 "R3" H 6900 3430 50  0000 C CNN
-F 1 "1k" H 6900 3350 50  0000 C CNN
-F 2 "" H 6900 3280 30  0000 C CNN
-F 3 "" V 6900 3350 30  0000 C CNN
-	1    6850 3300
-	0    1    1    0
-$EndComp
 Wire Wire Line
 	5300 3100 5750 3100
@@
 	6500 3200 6900 3200
 $Comp
-L C C1
-U 1 1 56A9B72C
-P 6100 2700
-F 0 "C1" H 6125 2800 50  0000 L CNN
-F 1 "100n" H 6125 2600 50  0000 L CNN
-F 2 "" H 6138 2550 30  0000 C CNN
-F 3 "" H 6100 2700 60  0000 C CNN
-	1    6100 2700
-	0    1    1    0
-$EndComp
-$Comp
-L GND #PWR01
+L GND #PWR2
 U 1 1 56A9B75D
 P 5450 3600
-F 0 "#PWR01" H 5450 3350 50  0001 C CNN
+F 0 "#PWR2" H 5450 3350 50  0001 C CNN
 F 1 "GND" H 5450 3450 50  0000 C CNN
 F 2 "" H 5450 3600 50  0000 C CNN
@@
 $EndComp
 $Comp
-L GND #PWR02
+L GND #PWR1
 U 1 1 56A9B7DC
 P 4800 4000
-F 0 "#PWR02" H 4800 3750 50  0001 C CNN
+F 0 "#PWR1" H 4800 3750 50  0001 C CNN
 F 1 "GND" H 4800 3850 50  0000 C CNN
 F 2 "" H 4800 4000 50  0000 C CNN
@@
 $EndComp
 $Comp
-L GND #PWR03
+L GND #PWR3
 U 1 1 56A9B7F9
 P 6900 3500
-F 0 "#PWR03" H 6900 3250 50  0001 C CNN
+F 0 "#PWR3" H 6900 3250 50  0001 C CNN
 F 1 "GND" H 6900 3350 50  0000 C CNN
 F 2 "" H 6900 3500 50  0000 C CNN
@@
 Wire Wire Line
 	6650 2350 6650 3200
-$Comp
-L R-RESCUE-Integrator R4
-U 1 1 56B2EBCB
-P 6050 2400
-F 0 "R4" H 6100 2530 50  0000 C CNN
-F 1 "100k" H 6100 2450 50  0000 C CNN
-F 2 "" H 6100 2380 30  0000 C CNN
-F 3 "" V 6100 2450 30  0000 C CNN
-	1    6050 2400
-	1    0    0    -1
-$EndComp
 Wire Wire Line
 	5950 2350 5600 2350
@@
 Connection ~ 4850 2950
 Connection ~ 6800 3050
+Text Notes 5050 2900 0    60   ~ 0
+10k
+Text Notes 5250 3700 0    60   ~ 0
+1k\n
+Text Notes 6300 2600 0    60   ~ 0
+100n
+Text Notes 5950 2150 0    60   ~ 0
+100k\n
+Text Notes 7100 3350 0    60   ~ 0
+1k
+$Comp
+L resistor R1
+U 1 1 5E68C500
+P 5100 3150
+F 0 "R1" H 5150 3280 50  0000 C CNN
+F 1 "10k" H 5150 3100 50  0000 C CNN
+F 2 "" H 5150 3130 30  0000 C CNN
+F 3 "" V 5150 3200 30  0000 C CNN
+	1    5100 3150
+	1    0    0    -1
+$EndComp
+$Comp
+L resistor R2
+U 1 1 5E68C560
+P 5400 3400
+F 0 "R2" H 5450 3530 50  0000 C CNN
+F 1 "1k" H 5450 3350 50  0000 C CNN
+F 2 "" H 5450 3380 30  0000 C CNN
+F 3 "" V 5450 3450 30  0000 C CNN
+	1    5400 3400
+	0    1    1    0
+$EndComp
+$Comp
+L resistor R3
+U 1 1 5E68C5B3
+P 6150 2300
+F 0 "R3" H 6200 2430 50  0000 C CNN
+F 1 "100k" H 6200 2250 50  0000 C CNN
+F 2 "" H 6200 2280 30  0000 C CNN
+F 3 "" V 6200 2350 30  0000 C CNN
+	1    6150 2300
+	-1   0    0    1
+$EndComp
+$Comp
+L capacitor C1
+U 1 1 5E68C612
+P 6100 2700
+F 0 "C1" H 6125 2800 50  0000 L CNN
+F 1 "100n" H 6125 2600 50  0000 L CNN
+F 2 "" H 6138 2550 30  0000 C CNN
+F 3 "" H 6100 2700 60  0000 C CNN
+	1    6100 2700
+	0    1    1    0
+$EndComp
+$Comp
+L resistor R4
+U 1 1 5E68C664
+P 6950 3400
+F 0 "R4" H 7000 3530 50  0000 C CNN
+F 1 "1k" H 7000 3350 50  0000 C CNN
+F 2 "" H 7000 3380 30  0000 C CNN
+F 3 "" V 7000 3450 30  0000 C CNN
+	1    6950 3400
+	0    -1   -1   0
+$EndComp
 $EndSCHEMATC
