File: Examples/Integrator_LM_741/Integrator_LM_741.sch (KiCad schematic (older format))
At the start: 11 parts, among them U1 plot_v1, U2 plot_v1, X1 lm_741

Commit message: part2/3 - .pro cleanup
Parts:
- v2, v3: symbol DC -> DC-RESCUE-Integrator_LM_741
Other:
- moved on the sheet: C1, R1, R2, R3, R4, U1, U2, X1, v1
