File: Examples/JK_Flipflop/JK_Flipflop.sch (KiCad schematic (older format))
At the start: 17 parts, among them U1 plot_v1, U10 adc_bridge_1, U2 plot_v1, U3 plot_v1, U4 plot_v1, U5 plot_v1, U6 adc_bridge_3, U7 dac_bridge_2, U8 adc_bridge_1, U9 d_jkff

Commit message: common code for Win and Linux, merged py2 changes
Parts:
- R1, R2: symbol R -> R-RESCUE-JK_Flipflop
Changed lines of the file:
@@
 EESchema Schematic File Version 2
+LIBS:JK_Flipflop-rescue
 LIBS:eSim_Analog
 LIBS:eSim_Devices
@@
 LIBS:74xx
 LIBS:cmos4000
+LIBS:JK_Flipflop-cache
 EELAYER 25 0
 EELAYER END
@@
 $EndComp
 $Comp
-L R R1
+L R-RESCUE-JK_Flipflop R1
 U 1 1 56D58F73
 P 9300 3200
@@
 $EndComp
 $Comp
-L R R2
+L R-RESCUE-JK_Flipflop R2
 U 1 1 56D58FBB
 P 9300 4000

Commit message: part2/3 - .pro cleanup
Parts:
- v1, v3, v4, v5: symbol DC -> DC-RESCUE-JK_Flipflop
Changed lines of the file:
@@
 LIBS:contrib
 LIBS:power
-LIBS:device
 LIBS:transistors
 LIBS:conn
-LIBS:linear
 LIBS:regul
 LIBS:74xx
@@
 $EndDescr
 $Comp
-L DC v1
+L DC-RESCUE-JK_Flipflop v1
 U 1 1 56D58CB2
 P 2400 3550
@@
 $EndComp
 $Comp
-L DC v3
+L DC-RESCUE-JK_Flipflop v3
 U 1 1 56D58D84
 P 3800 4350
@@
 $EndComp
 $Comp
-L DC v4
+L DC-RESCUE-JK_Flipflop v4
 U 1 1 56D5977A
 P 7300 1600
@@
 $EndComp
 $Comp
-L DC v5
+L DC-RESCUE-JK_Flipflop v5
 U 1 1 56D59898
 P 7300 5450
