File: Examples/Zener_Characteristic/Zener_Characteristic.sch (KiCad schematic (older format))
At the start: 5 parts, among them U1 zener, U2 plot_i2, U3 plot_v1

Commit message: changes in examples' .pro
Parts:
- v1: symbol DC -> DC-RESCUE-Zener_Characteristic
Changed lines of the file:
@@
 EESchema Schematic File Version 2
+LIBS:Zener_Characteristic-rescue
 LIBS:eSim_Analog
 LIBS:eSim_Devices
@@
 LIBS:contrib
 LIBS:power
-LIBS:device
 LIBS:transistors
 LIBS:conn
-LIBS:linear
 LIBS:regul
 LIBS:74xx
 LIBS:cmos4000
+LIBS:Zener_Characteristic-cache
 EELAYER 25 0
 EELAYER END
@@
 $EndDescr
 $Comp
-L DC v1
+L DC-RESCUE-Zener_Characteristic v1
 U 1 1 56C6E03A
 P 5350 3750
