File: Examples/FullwaveRectifier_SCR/scr.sch (KiCad schematic (older format))
At the start: 10 parts, among them U1 aswitch, U2 PORT

Commit message: SCR's .pro fixed
Parts:
- v1, v2: symbol dc -> dc-RESCUE-scr
Changed lines of the file:
@@
 EESchema Schematic File Version 2
+LIBS:scr-rescue
 LIBS:eSim_Analog
 LIBS:eSim_Devices
@@
 LIBS:eSim_User
 LIBS:power
-LIBS:device
 LIBS:transistors
 LIBS:conn
-LIBS:linear
 LIBS:regul
 LIBS:74xx
@@
 $EndComp
 $Comp
-L dc v1
+L dc-RESCUE-scr v1
 U 1 1 565DBF58
 P 3600 3700
@@
 $EndComp
 $Comp
-L dc v2
+L dc-RESCUE-scr v2
 U 1 1 565DC066
 P 5550 3000
