File: library/SubcircuitLibrary/4to16_demux/5_and.sch (KiCad schematic (older format))
At the start: 4 parts, among them U1 PORT, U2 d_and, U3 d_and, X1 3_and

Commit message: .pro changes in Subcircuits
Parts:
- X1: symbol 3_and -> 3_and-RESCUE-5_and
Changed lines of the file:
@@
 EESchema Schematic File Version 2
+LIBS:5_and-rescue
 LIBS:cypress
 LIBS:siliconi
@@
 LIBS:eSim_Plot
 LIBS:eSim_Power
-LIBS:eSim_PSpice
 LIBS:eSim_Sources
 LIBS:eSim_Subckt
@@
 $EndDescr
 $Comp
-L 3_and X1
+L 3_and-RESCUE-5_and X1
 U 1 1 5C9A2741
 P 3800 3350
