File: library/SubcircuitLibrary/74153/4_and.sch (KiCad schematic (older format))
At the start: 3 parts, among them U1 PORT, U2 d_and, X1 3_and

Commit message: .pro changes in Subcircuits
Parts:
- X1: symbol 3_and -> 3_and-RESCUE-4_and
Changed lines of the file:
@@
 EESchema Schematic File Version 2
+LIBS:4_and-rescue
 LIBS:texas
 LIBS:intel
@@
 LIBS:eSim_Plot
 LIBS:eSim_Power
-LIBS:eSim_PSpice
 LIBS:eSim_Sources
 LIBS:eSim_Subckt
 LIBS:eSim_User
+LIBS:4_and-cache
 EELAYER 25 0
 EELAYER END
@@
 $EndDescr
 $Comp
-L 3_and X1
+L 3_and-RESCUE-4_and X1
 U 1 1 5C9A2915
 P 3700 3500
