File: library/SubcircuitLibrary/74153/74153.sch (KiCad schematic (older format))
At the start: 15 parts, among them U1 PORT, U2 d_inverter, U3 d_inverter, U34 d_inverter, U35 d_inverter, X1 4_OR, X10 4_and, X2 4_OR, X3 4_and, X4 4_and, X5 4_and, X6 4_and, X7 4_and, X8 4_and, X9 4_and

Commit message: .pro changes in Subcircuits
Parts:
- X1, X2: symbol 4_OR -> 4_OR-RESCUE-74153
- X10, X3, X4, X5, X6, X7, X8, X9: symbol 4_and -> 4_and-RESCUE-74153
Changed lines of the file:
@@
 EESchema Schematic File Version 2
+LIBS:74153-rescue
 LIBS:power
-LIBS:device
+LIBS:eSim_User
 LIBS:texas
 LIBS:intel
@@
 LIBS:eSim_Plot
 LIBS:eSim_Power
-LIBS:eSim_PSpice
+LIBS:eSim_Subckt
 LIBS:eSim_Sources
-LIBS:eSim_User
-LIBS:eSim_Subckt
 LIBS:74153-cache
 EELAYER 25 0
@@
 YB
 $Comp
-L 4_and X8
+L 4_and-RESCUE-74153 X8
 U 1 1 5C9D0C22
 P 2750 3050
@@
 $EndComp
 $Comp
-L 4_and X9
+L 4_and-RESCUE-74153 X9
 U 1 1 5C9D0CA2
 P 2750 3600
@@
 $EndComp
 $Comp
-L 4_and X4
+L 4_and-RESCUE-74153 X4
 U 1 1 5C9D0D16
 P 2700 4200
@@
 $EndComp
 $Comp
-L 4_and X10
+L 4_and-RESCUE-74153 X10
 U 1 1 5C9D0D93
 P 2750 4700
@@
 $EndComp
 $Comp
-L 4_and X5
+L 4_and-RESCUE-74153 X5
 U 1 1 5C9D182A
 P 2700 5700
@@
 $EndComp
 $Comp
-L 4_and X6
+L 4_and-RESCUE-74153 X6
 U 1 1 5C9D1830
 P 2700 6250
@@
 $EndComp
 $Comp
-L 4_and X3
+L 4_and-RESCUE-74153 X3
 U 1 1 5C9D1836
 P 2650 6850
@@
 $EndComp
 $Comp
-L 4_and X7
+L 4_and-RESCUE-74153 X7
 U 1 1 5C9D183C
 P 2700 7350
@@
 	3750 6450 3750 6400
 $Comp
-L 4_OR X1
+L 4_OR-RESCUE-74153 X1
 U 1 1 5C9D22F7
 P 2150 8400
@@
 	4650 5400 5550 5400
 $Comp
-L 4_OR X2
+L 4_OR-RESCUE-74153 X2
 U 1 1 5C9D28DE
 P 2250 5750
