File: library/SubcircuitLibrary/74157/74157.sch (KiCad schematic (older format))
At the start: 15 parts, among them U1 PORT, U2 d_inverter, U20 d_or, U21 d_or, U22 d_or, U23 d_or, U3 d_inverter, X1 3_and, X2 3_and, X3 3_and, X4 3_and, X5 3_and, X6 3_and, X7 3_and, X8 3_and

Commit message: .pro changes in Subcircuits
Parts:
- X1, X2, X3, X4, X5, X6, X7, X8: symbol 3_and -> 3_and-RESCUE-74157
Changed lines of the file:
@@
 EESchema Schematic File Version 2
+LIBS:74157-rescue
 LIBS:power
 LIBS:intel
@@
 LIBS:eSim_Plot
 LIBS:eSim_Power
-LIBS:eSim_PSpice
+LIBS:eSim_Subckt
 LIBS:eSim_Sources
 LIBS:eSim_User
-LIBS:eSim_Subckt
 LIBS:74157-cache
 EELAYER 25 0
@@
 Connection ~ 3450 5700
 $Comp
-L 3_and X2
+L 3_and-RESCUE-74157 X2
 U 1 1 5C9D0110
 P 3450 2400
@@
 $EndComp
 $Comp
-L 3_and X3
+L 3_and-RESCUE-74157 X3
 U 1 1 5C9D01B8
 P 3450 2900
@@
 $EndComp
 $Comp
-L 3_and X4
+L 3_and-RESCUE-74157 X4
 U 1 1 5C9D0222
 P 3450 3350
@@
 $EndComp
 $Comp
-L 3_and X5
+L 3_and-RESCUE-74157 X5
 U 1 1 5C9D0289
 P 3450 3850
@@
 $EndComp
 $Comp
-L 3_and X6
+L 3_and-RESCUE-74157 X6
 U 1 1 5C9D0361
 P 3450 4650
@@
 $EndComp
 $Comp
-L 3_and X7
+L 3_and-RESCUE-74157 X7
 U 1 1 5C9D0367
 P 3450 5150
@@
 $EndComp
 $Comp
-L 3_and X1
+L 3_and-RESCUE-74157 X1
 U 1 1 5C9D036D
 P 3400 5600
@@
 $EndComp
 $Comp
-L 3_and X8
+L 3_and-RESCUE-74157 X8
 U 1 1 5C9D0373
 P 3450 6100
