File: library/SubcircuitLibrary/7485/7485.sch (KiCad schematic (older format))
At the start: 32 parts, among them U1 PORT, U10 d_and, U11 d_and, U12 d_and, U13 d_and, U14 d_nor, U15 d_nor, U16 d_nor, U17 d_nor, U18 d_and, U19 d_and, U2 d_nand, U3 d_nand, U4 d_nand, U5 d_nand, U6 d_and, U7 d_and, U8 d_and, U9 d_and, X1 c_gate, X10 5_and, X11 5_and, X12 3_and, X13 5_and, X2 c_gate, X3 4_and, X4 5_and, X5 5_and, X6 5_and, X7 4_and, X8 3_and, X9 5_and

Commit message: .pro changes in Subcircuits
Parts:
- X10, X11, X13, X4, X5, X6, X9: symbol 5_and -> 5_and-RESCUE-7485
- X12, X8: symbol 3_and -> 3_and-RESCUE-7485
- X3, X7: symbol 4_and -> 4_and-RESCUE-7485
Connections:
- wire segments 242 -> 182
Changed lines of the file:
@@
 EESchema Schematic File Version 2
+LIBS:7485-rescue
 LIBS:power
 LIBS:texas
@@
 LIBS:eSim_Plot
 LIBS:eSim_Power
-LIBS:eSim_PSpice
+LIBS:eSim_Subckt
 LIBS:eSim_Sources
 LIBS:eSim_User
-LIBS:eSim_Subckt
 LIBS:7485-cache
 EELAYER 25 0
@@
 $EndComp
 $Comp
-L 3_and X12
+L 3_and-RESCUE-7485 X12
 U 1 1 5C9A2DC4
 P 6050 1650
@@
 $EndComp
 $Comp
-L 4_and X7
+L 4_and-RESCUE-7485 X7
 U 1 1 5C9A2EB7
 P 5450 2750
@@
 $EndComp
 $Comp
-L 5_and X9
+L 5_and-RESCUE-7485 X9
 U 1 1 5C9A2F2E
 P 5650 3050
@@
 $EndComp
 $Comp
-L 5_and X10
+L 5_and-RESCUE-7485 X10
 U 1 1 5C9A2F95
 P 5650 3600
@@
 $EndComp
 $Comp
-L 5_and X11
+L 5_and-RESCUE-7485 X11
 U 1 1 5C9A3164
 P 5650 4150
@@
 $EndComp
 $Comp
-L 5_and X13
+L 5_and-RESCUE-7485 X13
 U 1 1 5C9A31B3
 P 7550 4850
@@
 $EndComp
 $Comp
-L 3_and X8
+L 3_and-RESCUE-7485 X8
 U 1 1 5C9A3303
 P 5500 6250
@@
 $EndComp
 $Comp
-L 4_and X3
+L 4_and-RESCUE-7485 X3
 U 1 1 5C9A3309
 P 4900 5150
@@
 $EndComp
 $Comp
-L 5_and X6
+L 5_and-RESCUE-7485 X6
 U 1 1 5C9A330F
 P 5100 4850
@@
 $EndComp
 $Comp
-L 5_and X5
+L 5_and-RESCUE-7485 X5
 U 1 1 5C9A3315
 P 5100 4300
@@
 $EndComp
 $Comp
-L 5_and X4
+L 5_and-RESCUE-7485 X4
 U 1 1 5C9A331B
 P 5100 3750
@@
 	3600 1400 3600 1550
 Wire Wire Line
-	2700 1000 2700 1200
-Wire Wire Line
-	2700 1200 2700 1400
-Wire Wire Line
-	2700 1400 2700 1500
-Wire Wire Line
-	2700 1500 2700 4700
+	2700 1000 2700 4700
 Wire Wire Line
 	2700 1600 1550 1600
 Wire Wire Line
-	1550 1600 1550 1450
-Wire Wire Line
-	1100 1450 1500 1450
-Wire Wire Line
-	1500 1450 1550 1450
-Wire Wire Line
-	1550 1450 1650 1450
-Wire Wire Line
-	1100 1350 1400 1350
-Wire Wire Line
-	1400 1350 1550 1350
-Wire Wire Line
-	1550 1350 1650 1350
+	1550 1450 1550 1600
+Wire Wire Line
+	1100 1450 1650 1450
+Wire Wire Line
+	1100 1350 1650 1350
 Wire Wire Line
 	1550 1350 1550 1100
@@
 	3700 2800 3700 2950
 Wire Wire Line
-	2800 2000 2800 2600
-Wire Wire Line
-	2800 2600 2800 2800
-Wire Wire Line
-	2800 2800 2800 2900
-Wire Wire Line
-	2800 2900 2800 4600
+	2800 2000 2800 4600
 Wire Wire Line
 	2800 3000 1650 3000
 Wire Wire Line
-	1650 3000 1650 2850
-Wire Wire Line
-	1200 2850 1600 2850
-Wire Wire Line
-	1600 2850 1650 2850
-Wire Wire Line
-	1650 2850 1750 2850
-Wire Wire Line
-	1200 2750 1450 2750
-Wire Wire Line
-	1450 2750 1650 2750
-Wire Wire Line
-	1650 2750 1750 2750
+	1650 2850 1650 3000
+Wire Wire Line
+	1200 2850 1750 2850
+Wire Wire Line
+	1200 2750 1750 2750
 Wire Wire Line
 	1650 2750 1650 2500
@@
 	4050 5150 4050 5300
 Wire Wire Line
-	3150 4950 3150 5000
-Wire Wire Line
-	3150 5000 3150 5150
-Wire Wire Line
-	3150 5150 3150 5250
-Wire Wire Line
-	3150 5250 3150 5850
+	3150 4950 3150 5850
 Wire Wire Line
 	3150 5350 2000 5350
 Wire Wire Line
-	2000 5350 2000 5200
-Wire Wire Line
-	1250 5200 1500 5200
-Wire Wire Line
-	1500 5200 2000 5200
-Wire Wire Line
-	2000 5200 2100 5200
-Wire Wire Line
-	1250 5100 1800 5100
-Wire Wire Line
-	1800 5100 2000 5100
-Wire Wire Line
-	2000 5100 2100 5100
+	2000 5200 2000 5350
+Wire Wire Line
+	1250 5200 2100 5200
+Wire Wire Line
+	1250 5100 2100 5100
 Wire Wire Line
 	2000 5100 2000 4850
@@
 	3850 3950 3850 4100
 Wire Wire Line
-	2950 3200 2950 3750
-Wire Wire Line
-	2950 3750 2950 3950
-Wire Wire Line
-	2950 3950 2950 4050
-Wire Wire Line
-	2950 4050 2950 4350
+	2950 3200 2950 4350
 Wire Wire Line
 	2950 4150 1800 4150
 Wire Wire Line
-	1800 4150 1800 4000
-Wire Wire Line
-	1350 4000 1750 4000
-Wire Wire Line
-	1750 4000 1800 4000
-Wire Wire Line
-	1800 4000 1900 4000
-Wire Wire Line
-	1200 3900 1600 3900
-Wire Wire Line
-	1600 3900 1800 3900
-Wire Wire Line
-	1800 3900 1900 3900
+	1800 4000 1800 4150
+Wire Wire Line
+	1350 4000 1900 4000
+Wire Wire Line
+	1200 3900 1900 3900
 Wire Wire Line
 	1800 3900 1800 3650
@@
 	5100 6550 5950 6550
 Wire Wire Line
-	5100 1350 5100 1700
-Wire Wire Line
-	5100 1700 5100 2150
-Wire Wire Line
-	5100 2150 5100 2500
-Wire Wire Line
-	5100 2500 5100 3050
-Wire Wire Line
-	5100 3050 5100 3750
-Wire Wire Line
-	5100 3750 5100 4850
-Wire Wire Line
-	5100 4850 5100 5400
-Wire Wire Line
-	5100 5400 5100 5750
-Wire Wire Line
-	5100 5750 5100 6300
-Wire Wire Line
-	5100 6300 5100 6550
-Wire Wire Line
-	4500 1350 5100 1350
-Wire Wire Line
-	5100 1350 6500 1350
+	5100 1350 5100 6550
+Wire Wire Line
+	4500 1350 6500 1350
 Wire Wire Line
 	1500 1450 1500 900
@@
 	6500 1800 5250 1800
 Wire Wire Line
-	5250 1800 5250 2250
-Wire Wire Line
-	5250 2250 5250 2600
-Wire Wire Line
-	5250 2600 5250 2750
-Wire Wire Line
-	5250 2750 5250 3150
-Wire Wire Line
-	5250 3150 5250 3850
-Wire Wire Line
-	5250 3850 5250 4750
-Wire Wire Line
-	5250 4750 5250 5300
-Wire Wire Line
-	5250 5300 5250 5650
-Wire Wire Line
-	5250 5650 5250 6100
+	5250 1800 5250 6100
 Wire Wire Line
 	5250 2750 4600 2750
@@
 	6500 2350 5350 2350
 Wire Wire Line
-	5350 2350 5350 2700
-Wire Wire Line
-	5350 2700 5350 3200
-Wire Wire Line
-	5350 3200 5350 3900
-Wire Wire Line
-	5350 3900 5350 4050
-Wire Wire Line
-	5350 4050 5350 4650
-Wire Wire Line
-	5350 4650 5350 5200
-Wire Wire Line
-	5350 5200 5350 5550
+	5350 2350 5350 5550
 Wire Wire Line
 	5350 3900 4750 3900
@@
 	6500 2800 5450 2800
 Wire Wire Line
-	5450 2800 5450 3350
-Wire Wire Line
-	5450 3350 5450 4150
-Wire Wire Line
-	5450 4150 5450 4550
-Wire Wire Line
-	5450 4550 5450 5100
-Wire Wire Line
-	4950 5100 5450 5100
-Wire Wire Line
-	5450 5100 5950 5100
+	5450 2800 5450 5100
+Wire Wire Line
+	4950 5100 5950 5100
 Wire Wire Line
 	6500 2900 5550 2900
@@
 Connection ~ 5450 3350
 Wire Wire Line
-	4800 3450 5950 3450
-Wire Wire Line
-	5950 3450 6500 3450
-Wire Wire Line
-	4800 3450 4800 3400
-Wire Wire Line
-	4800 3400 2600 3400
-Wire Wire Line
-	2050 3400 1050 3400
-Wire Wire Line
-	5950 3450 5950 3950
-Wire Wire Line
-	5950 3950 5950 4450
+	4800 3450 6500 3450
+Wire Wire Line
+	4800 3400 4800 3450
+Wire Wire Line
+	1050 3400 4800 3400
+Wire Wire Line
+	5950 3450 5950 4450
 Connection ~ 5950 3450
 Wire Wire Line
@@
 Text Notes 9900 3400 0    60   ~ 12
 Outputs
-Wire Wire Line
-	2600 3400 2050 3400
 $EndSCHEMATC
