File: library/SubcircuitLibrary/7485/c_gate.sch (KiCad schematic (older format))
At the start: 9 parts, among them U1 PORT, U2 d_inverter, U3 d_inverter, U4 d_inverter, U5 d_inverter, U6 d_inverter, U7 d_inverter, U8 d_and, X1 5_and

Commit message: .pro changes in Subcircuits
Parts:
- X1: symbol 5_and -> 5_and-RESCUE-c_gate
Changed lines of the file:
@@
 EESchema Schematic File Version 2
+LIBS:c_gate-rescue
 LIBS:texas
 LIBS:intel
@@
 LIBS:eSim_Plot
 LIBS:eSim_Power
-LIBS:eSim_PSpice
 LIBS:eSim_Sources
 LIBS:eSim_Subckt
@@
 $EndDescr
 $Comp
-L 5_and X1
+L 5_and-RESCUE-c_gate X1
 U 1 1 5C9A2B0B
 P 3300 3750
